File: Breakouts/4051_breakout_smd/4051_breakout.sch (KiCad schematic (older format))
At the start: 6 parts, among them J1 Conn_01x08, J2 Conn_01x08, U1 4051, U2 4051

Commit message: 4051 breakout updates (forgot what exactly)
Parts:
- C1: symbol C_Small -> Device:C_Small
- J1, J2: symbol Conn_01x08 -> conn:Conn_01x08
- R1: symbol R_Small -> Device:R_Small
- U1, U2: symbol 4051 -> cmos4000:4051
Changed lines of the file:
@@
-EESchema Schematic File Version 2
-LIBS:power
-LIBS:device
-LIBS:switches
-LIBS:relays
-LIBS:motors
-LIBS:transistors
-LIBS:conn
-LIBS:linear
-LIBS:regul
-LIBS:74xx
-LIBS:cmos4000
-LIBS:adc-dac
-LIBS:memory
-LIBS:xilinx
-LIBS:microcontrollers
-LIBS:dsp
-LIBS:microchip
-LIBS:analog_switches
-LIBS:motorola
-LIBS:texas
-LIBS:intel
-LIBS:audio
-LIBS:interface
-LIBS:digital-audio
-LIBS:philips
-LIBS:display
-LIBS:cypress
-LIBS:siliconi
-LIBS:opto
-LIBS:atmel
-LIBS:contrib
-LIBS:valves
-EELAYER 25 0
+EESchema Schematic File Version 4
+LIBS:4051_breakout-cache
+EELAYER 29 0
 EELAYER END
 $Descr A4 11693 8268
@@
 $EndDescr
 $Comp
-L 4051 U1
+L cmos4000:4051 U1
 U 1 1 5CB4578E
 P 5050 3050
@@
 $EndComp
 $Comp
-L 4051 U2
+L cmos4000:4051 U2
 U 1 1 5CB45804
 P 5050 3050
@@
 Connection ~ 4350 3050
 Connection ~ 4350 3150
-Connection ~ 4350 3350
-Connection ~ 4350 3450
-Connection ~ 4350 3550
-Connection ~ 4350 3650
-Connection ~ 5750 3550
-Connection ~ 5750 2450
 $Comp
-L VSS #PWR01
+L power:VSS #PWR01
 U 1 1 5CB458C9
 P 3400 3100
@@
 $EndComp
 $Comp
-L VDD #PWR02
+L power:VDD #PWR02
 U 1 1 5CB458E3
 P 3400 3800
@@
 $EndComp
 $Comp
-L Conn_01x08 J2
+L conn:Conn_01x08 J2
 U 1 1 5CB45923
 P 4150 2850
@@
 $EndComp
 $Comp
-L Conn_01x08 J1
+L conn:Conn_01x08 J1
 U 1 1 5CB45973
 P 3200 3500
@@
 $EndComp
 $Comp
-L VSS #PWR03
+L power:VSS #PWR03
 U 1 1 5CB459BF
 P 5950 4150
@@
 $EndComp
 $Comp
-L C_Small C1
+L Device:C_Small C1
 U 1 1 5CB459D1
 P 5950 4050
@@
 $EndComp
 $Comp
-L VDD #PWR04
+L power:VDD #PWR04
 U 1 1 5CB45BE0
 P 5950 3950
@@
 $EndComp
 $Comp
-L R_Small R1
+L Device:R_Small R1
 U 1 1 5CB45D66
 P 4000 3250
@@
 $EndComp
 $Comp
-L VSS #PWR05
+L power:VSS #PWR05
 U 1 1 5CB45E66
 P 4000 3150
@@
 	1    0    0    -1
 $EndComp
-Connection ~ 4000 3350
 Text GLabel 4350 3650 0    60   Input ~ 0
 C
