File: Peripherals/pcf8574_dip_breakout/pcf8574_dip_breakout/pcf8574_dip_breakout.sch (KiCad schematic (older format))
At the start: 4 parts

Commit message: PCF8574 breakout - finished, need to double-check later
Parts:
- removed J?: Conn_01x09, symbol Connector_Generic:Conn_01x09
- added D1, D2, D3, D4, D5, D6, D7, D8: LED, LED_SMD:LED_0805_2012Metric_Pad1.15x1.40mm_HandSolder, symbol Device:LED_Small
- added J2: IO, Connector_PinHeader_2.54mm:PinHeader_1x10_P2.54mm_Vertical, symbol Connector_Generic:Conn_01x10
- added JP1: A2, pcf8574_dip_breakout:GS3_SMALL, symbol Jumper:Jumper_3_Open
- added JP2: A1, pcf8574_dip_breakout:GS3_SMALL, symbol Jumper:Jumper_3_Open
- added JP3: A0, pcf8574_dip_breakout:GS3_SMALL, symbol Jumper:Jumper_3_Open
- added R1: 10K, pcf8574_dip_breakout:R_0805_10K_HandSoldering, symbol Device:R_Small
- added R2, R3, R4, R5, R6, R7, R8, R9: 1K, pcf8574_dip_breakout:R_0805_10K_HandSoldering, symbol Device:R_Small
- C1: renamed from C?; footprint (none) -> pcf8574_dip_breakout:C_0805_100nF_HandSoldering
- J1: renamed from J?; footprint (none) -> Connector_PinHeader_2.54mm:PinHeader_1x05_P2.54mm_Vertical
- U1: renamed from U?; footprint (none) -> Package_DIP:DIP-16_W7.62mm_LongPads
Connections:
- net A0: now also JP1.2 (C)
- net A1: now also JP2.2 (C)
- net A2: now also JP3.2 (C)
- net GND: now also C1.2, J2.10 (Pin_10), JP1.3 (B), JP2.3 (B), JP3.3 (B)
- net INT: now also R1.2
- net O0: now also D1.1 (K), J2.2 (Pin_2)
- net O1: now also D2.1 (K), J2.3 (Pin_3)
- net O2: now also D3.1 (K), J2.4 (Pin_4)
- net O3: now also D4.1 (K), J2.5 (Pin_5)
- net O4: now also D5.1 (K), J2.6 (Pin_6)
- net O5: now also D6.1 (K), J2.7 (Pin_7)
- net O6: now also D7.1 (K), J2.8 (Pin_8)
- net O7: now also D8.1 (K), J2.9 (Pin_9)
- net VCC: now also C1.1, J2.1 (Pin_1), JP1.1 (A), JP2.1 (A), JP3.1 (A), R1.1, R2.1, R3.1, R4.1, R5.1, R6.1, R7.1, R8.1, R9.1
- new net: D1.2 (A), R2.2
- new net: D2.2 (A), R3.2
- new net: D3.2 (A), R4.2
- new net: D4.2 (A), R5.2
- new net: D5.2 (A), R6.2
- new net: D6.2 (A), R7.2
- new net: D7.2 (A), R8.2
- new net: D8.2 (A), R9.2
Other:
- moved on the sheet: C1, J1
