File: Reverse-engineering/keyboard_whiz/keyboard_whiz.sch (KiCad schematic (older format))
At the start: 27 parts, among them J1 I2C, J2 0.5mm, J3 0.8mm, J4 1mm, J5 Raspberry_Pi_2_3, SW1 32-39 switch, U1 0x21, U2 0x22

Commit message: Latest revision of Keyboard Whiz - one that went into v1 production
Parts:
- removed SW1: 32-39 switch, Connector_PinHeader_2.54mm:PinHeader_2x08_P2.54mm_Vertical, symbol Connector_Generic:Conn_02x08_Odd_Even
- added D2: 1N4148, Diode_SMD:D_MiniMELF, symbol Device:D_Small
- J2, J3, J4: symbol Connector_Generic_MountingPin:Conn_01x40_MountingPin -> Connector_Generic_MountingPin:Conn_01x32_MountingPin
Connections:
- net INT: now also D2.2 (A)
- removed net C32: J2.33 (Pin_33), J3.33 (Pin_33), J4.33 (Pin_33)
- removed net C33: J2.34 (Pin_34), J3.34 (Pin_34), J4.34 (Pin_34)
- removed net C34: J2.35 (Pin_35), J3.35 (Pin_35), J4.35 (Pin_35)
- removed net C35: J2.36 (Pin_36), J3.36 (Pin_36), J4.36 (Pin_36)
- removed net C36: J2.37 (Pin_37), J3.37 (Pin_37), J4.37 (Pin_37)
- removed net C37: J2.38 (Pin_38), J3.38 (Pin_38), J4.38 (Pin_38)
- removed net C38: J2.39 (Pin_39), J3.39 (Pin_39), J4.39 (Pin_39)
- removed net C39: J2.40 (Pin_40), J3.40 (Pin_40), J4.40 (Pin_40)
- net INTO renamed INTO1
- net INTO1: no longer U2.19 (INTB), U2.20 (INTA)
- new net INTO2: D2.1 (K), U2.19 (INTB), U2.20 (INTA)
