File: Atmel/fan_controller/fan_controller.sch (KiCad schematic (older format))
At the start: 24 parts, among them J1 I2C, J2 FAN, J3 POT, J4 AVR-ISP-6, J5 PWR, J6 I2C_PWR, Q1 Q_PMOS_GSD, Q2 BC817, U1 LM1117-5.0, U2 ATtiny45-20P, U3 ATtiny13V-10S

Commit message: Fixing the SOT23 footprint so that BC817 works properly, adding a TACH pullup, rerouting the board to fit it and moving silkscreen stuff around
Parts:
- removed Q2: BC817, Package_TO_SOT_SMD:SOT-23, symbol Device:Q_NPN_BCE
- added Q2: BC817, Package_TO_SOT_SMD:SOT-23, symbol Device:Q_NPN_BEC
- added R6: 10K, Resistor_SMD:R_0805_2012Metric, symbol Device:R_Small
- U2: symbol MCU_Microchip_ATtiny:ATtiny45-20P -> fan_controller-rescue:ATtiny45-20P-MCU_Microchip_ATtiny
- U3: symbol MCU_Microchip_ATtiny:ATtiny13V-10S -> fan_controller-rescue:ATtiny13V-10S-MCU_Microchip_ATtiny
Connections:
- net GND: now also Q2.2 (E)
- net TACH: now also R6.2
- net VCC: now also R6.1
- net at Q1.1 (G), R1.2: now also Q2.3 (C)
- net at R2.2: now also Q2.1 (B)
Other:
- moved on the sheet: C1, C2, U1
Changed lines of the file:
@@
 L Device:C_Small C2
 U 1 1 61593F2C
-P 8850 1550
-F 0 "C2" H 8942 1596 50  0000 L CNN
-F 1 "100nF" H 8942 1505 50  0000 L CNN
-F 2 "Capacitor_SMD:C_0805_2012Metric" H 8850 1550 50  0001 C CNN
-F 3 "~" H 8850 1550 50  0001 C CNN
-	1    8850 1550
-	1    0    0    -1
-$EndComp
-$Comp
-L MCU_Microchip_ATtiny:ATtiny13V-10S U3
+P 9400 1550
+F 0 "C2" H 9492 1596 50  0000 L CNN
+F 1 "100nF" H 9492 1505 50  0000 L CNN
+F 2 "Capacitor_SMD:C_0805_2012Metric" H 9400 1550 50  0001 C CNN
+F 3 "~" H 9400 1550 50  0001 C CNN
+	1    9400 1550
+	1    0    0    -1
+$EndComp
+$Comp
+L fan_controller-rescue:ATtiny13V-10S-MCU_Microchip_ATtiny U3
 U 1 1 615959AF
 P 9750 4900
@@
 $EndComp
 $Comp
-L MCU_Microchip_ATtiny:ATtiny45-20P U2
+L fan_controller-rescue:ATtiny45-20P-MCU_Microchip_ATtiny U2
 U 1 1 615963D2
 P 9700 2900
@@
 L fan_controller-rescue:VCC #PWR0101
 U 1 1 6159841F
-P 8400 1450
-F 0 "#PWR0101" H 8400 1300 50  0001 C CNN
-F 1 "VCC" H 8417 1623 50  0000 C CNN
-F 2 "" H 8400 1450 50  0001 C CNN
-F 3 "" H 8400 1450 50  0001 C CNN
-	1    8400 1450
+P 8950 1450
+F 0 "#PWR0101" H 8950 1300 50  0001 C CNN
+F 1 "VCC" H 8967 1623 50  0000 C CNN
+F 2 "" H 8950 1450 50  0001 C CNN
+F 3 "" H 8950 1450 50  0001 C CNN
+	1    8950 1450
 	1    0    0    -1
 $EndComp
@@
 L fan_controller-rescue:GND #PWR0105
 U 1 1 615A102E
-P 8850 1650
-F 0 "#PWR0105" H 8850 1400 50  0001 C CNN
-F 1 "GND" H 8855 1477 50  0000 C CNN
-F 2 "" H 8850 1650 50  0001 C CNN
-F 3 "" H 8850 1650 50  0001 C CNN
-	1    8850 1650
+P 9400 1650
+F 0 "#PWR0105" H 9400 1400 50  0001 C CNN
+F 1 "GND" H 9405 1477 50  0000 C CNN
+F 2 "" H 9400 1650 50  0001 C CNN
+F 3 "" H 9400 1650 50  0001 C CNN
+	1    9400 1650
 	1    0    0    -1
 $EndComp
@@
 L Device:C_Small C1
 U 1 1 615A4CD5
-P 8400 1550
-F 0 "C1" H 8492 1596 50  0000 L CNN
-F 1 "100nF" H 8492 1505 50  0000 L CNN
-F 2 "Capacitor_SMD:C_0805_2012Metric" H 8400 1550 50  0001 C CNN
-F 3 "~" H 8400 1550 50  0001 C CNN
-	1    8400 1550
+P 8950 1550
+F 0 "C1" H 9042 1596 50  0000 L CNN
+F 1 "100nF" H 9042 1505 50  0000 L CNN
+F 2 "Capacitor_SMD:C_0805_2012Metric" H 8950 1550 50  0001 C CNN
+F 3 "~" H 8950 1550 50  0001 C CNN
+	1    8950 1550
 	1    0    0    -1
 $EndComp
@@
 L fan_controller-rescue:GND #PWR0106
 U 1 1 615A4CDF
-P 8400 1650
-F 0 "#PWR0106" H 8400 1400 50  0001 C CNN
-F 1 "GND" H 8405 1477 50  0000 C CNN
-F 2 "" H 8400 1650 50  0001 C CNN
-F 3 "" H 8400 1650 50  0001 C CNN
-	1    8400 1650
+P 8950 1650
+F 0 "#PWR0106" H 8950 1400 50  0001 C CNN
+F 1 "GND" H 8955 1477 50  0000 C CNN
+F 2 "" H 8950 1650 50  0001 C CNN
+F 3 "" H 8950 1650 50  0001 C CNN
+	1    8950 1650
 	1    0    0    -1
 $EndComp
@@
 L fan_controller-rescue:VCC #PWR0107
 U 1 1 615A7D7A
-P 9300 1300
-F 0 "#PWR0107" H 9300 1150 50  0001 C CNN
-F 1 "VCC" H 9317 1473 50  0000 C CNN
-F 2 "" H 9300 1300 50  0001 C CNN
-F 3 "" H 9300 1300 50  0001 C CNN
-	1    9300 1300
+P 9850 1300
+F 0 "#PWR0107" H 9850 1150 50  0001 C CNN
+F 1 "VCC" H 9867 1473 50  0000 C CNN
+F 2 "" H 9850 1300 50  0001 C CNN
+F 3 "" H 9850 1300 50  0001 C CNN
+	1    9850 1300
 	1    0    0    -1
 $EndComp
@@
 L fan_controller-rescue:GND #PWR0108
 U 1 1 615A83DB
-P 9600 1600
-F 0 "#PWR0108" H 9600 1350 50  0001 C CNN
-F 1 "GND" H 9605 1427 50  0000 C CNN
-F 2 "" H 9600 1600 50  0001 C CNN
-F 3 "" H 9600 1600 50  0001 C CNN
-	1    9600 1600
+P 10150 1600
+F 0 "#PWR0108" H 10150 1350 50  0001 C CNN
+F 1 "GND" H 10155 1427 50  0000 C CNN
+F 2 "" H 10150 1600 50  0001 C CNN
+F 3 "" H 10150 1600 50  0001 C CNN
+	1    10150 1600
 	1    0    0    -1
 $EndComp
@@
 L power:+5V #PWR0109
 U 1 1 615ADEA5
-P 9900 1300
-F 0 "#PWR0109" H 9900 1150 50  0001 C CNN
-F 1 "+5V" H 9915 1473 50  0000 C CNN
-F 2 "" H 9900 1300 50  0001 C CNN
-F 3 "" H 9900 1300 50  0001 C CNN
-	1    9900 1300
+P 10450 1300
+F 0 "#PWR0109" H 10450 1150 50  0001 C CNN
+F 1 "+5V" H 10465 1473 50  0000 C CNN
+F 2 "" H 10450 1300 50  0001 C CNN
+F 3 "" H 10450 1300 50  0001 C CNN
+	1    10450 1300
 	1    0    0    -1
 $EndComp
@@
 L Regulator_Linear:LM1117-5.0 U1
 U 1 1 615AFE6E
-P 9600 1300
-F 0 "U1" H 9550 1450 50  0000 C CNN
-F 1 "LM1117-5.0" H 9900 1000 50  0000 C CNN
-F 2 "Package_TO_SOT_SMD:SOT-223-3_TabPin2" H 9600 1300 50  0001 C CNN
-F 3 "http://www.ti.com/lit/ds/symlink/lm1117.pdf" H 9600 1300 50  0001 C CNN
-	1    9600 1300
+P 10150 1300
+F 0 "U1" H 10100 1450 50  0000 C CNN
+F 1 "LM1117-5.0" H 10450 1000 50  0000 C CNN
+F 2 "Package_TO_SOT_SMD:SOT-223-3_TabPin2" H 10150 1300 50  0001 C CNN
+F 3 "http://www.ti.com/lit/ds/symlink/lm1117.pdf" H 10150 1300 50  0001 C CNN
+	1    10150 1300
 	1    0    0    -1
 $EndComp
@@
 Wire Wire Line
 	7650 2700 7650 2650
-$Comp
-L Device:Q_NPN_BCE Q2
-U 1 1 615DEC38
-P 7550 3500
-F 0 "Q2" H 7741 3546 50  0000 L CNN
-F 1 "BC817" H 7741 3455 50  0000 L CNN
-F 2 "Package_TO_SOT_SMD:SOT-23" H 7750 3600 50  0001 C CNN
-F 3 "~" H 7550 3500 50  0001 C CNN
-	1    7550 3500
-	-1   0    0    -1
-$EndComp
 Wire Wire Line
 	7450 3300 7450 3200
@@
 L power:+5V #PWR0104
 U 1 1 61621802
-P 8850 1450
-F 0 "#PWR0104" H 8850 1300 50  0001 C CNN
-F 1 "+5V" H 8865 1623 50  0000 C CNN
-F 2 "" H 8850 1450 50  0001 C CNN
-F 3 "" H 8850 1450 50  0001 C CNN
-	1    8850 1450
+P 9400 1450
+F 0 "#PWR0104" H 9400 1300 50  0001 C CNN
+F 1 "+5V" H 9415 1623 50  0000 C CNN
+F 2 "" H 9400 1450 50  0001 C CNN
+F 3 "" H 9400 1450 50  0001 C CNN
+	1    9400 1450
 	1    0    0    -1
 $EndComp
@@
 	1    0    0    -1
 $EndComp
+$Comp
+L Device:R_Small R6
+U 1 1 616E6E98
+P 8550 1550
+F 0 "R6" H 8609 1596 50  0000 L CNN
+F 1 "10K" H 8609 1505 50  0000 L CNN
+F 2 "Resistor_SMD:R_0805_2012Metric" H 8550 1550 50  0001 C CNN
+F 3 "~" H 8550 1550 50  0001 C CNN
+	1    8550 1550
+	1    0    0    -1
+$EndComp
+$Comp
+L fan_controller-rescue:VCC #PWR0125
+U 1 1 616E7D14
+P 8550 1450
+F 0 "#PWR0125" H 8550 1300 50  0001 C CNN
+F 1 "VCC" H 8567 1623 50  0000 C CNN
+F 2 "" H 8550 1450 50  0001 C CNN
+F 3 "" H 8550 1450 50  0001 C CNN
+	1    8550 1450
+	1    0    0    -1
+$EndComp
+Text GLabel 8550 1650 0    50   Input ~ 0
+TACH
+$Comp
+L Device:Q_NPN_BEC Q2
+U 1 1 616F7FA8
+P 7550 3500
+F 0 "Q2" H 7741 3546 50  0000 L CNN
+F 1 "BC817" H 7741 3455 50  0000 L CNN
+F 2 "Package_TO_SOT_SMD:SOT-23" H 7750 3600 50  0001 C CNN
+F 3 "~" H 7550 3500 50  0001 C CNN
+	1    7550 3500
+	-1   0    0    -1
+$EndComp
 $EndSCHEMATC
