File: Power stuff/usb_power_switcher/usb_power_switcher.sch (KiCad schematic (older format))
At the start: 18 parts, among them J1 IN, J2 Conn_01x04, J3 OUT, J4 D+, J5 D-, J6 USB_OTG, Q1 Q_NPN_BEC, Q2 Q_PMOS_GSD

Commit message: Reloading the USB power switcher project files
Parts:
- D1, D2, D3: symbol LED -> usb_power_switcher-rescue:LED
- J1, J3: symbol USB_A -> usb_power_switcher-rescue:USB_A
- J2: symbol Conn_01x04 -> usb_power_switcher-rescue:Conn_01x04
- J4, J5: symbol GS2 -> usb_power_switcher-rescue:GS2
- J6: symbol USB_OTG -> usb_power_switcher-rescue:USB_OTG
- Q1: symbol Q_NPN_BEC -> usb_power_switcher-rescue:Q_NPN_BEC
- Q2: symbol Q_PMOS_GSD -> usb_power_switcher-rescue:Q_PMOS_GSD
- R1, R2, R3, R4, R5, R6, R7: symbol R_Small -> usb_power_switcher-rescue:R_Small
Changed lines of the file:
@@
-EESchema Schematic File Version 2
-LIBS:power
-LIBS:device
-LIBS:switches
-LIBS:relays
-LIBS:motors
-LIBS:transistors
-LIBS:conn
-LIBS:linear
-LIBS:regul
-LIBS:74xx
-LIBS:cmos4000
-LIBS:adc-dac
-LIBS:memory
-LIBS:xilinx
-LIBS:microcontrollers
-LIBS:dsp
-LIBS:microchip
-LIBS:analog_switches
-LIBS:motorola
-LIBS:texas
-LIBS:intel
-LIBS:audio
-LIBS:interface
-LIBS:digital-audio
-LIBS:philips
-LIBS:display
-LIBS:cypress
-LIBS:siliconi
-LIBS:opto
-LIBS:atmel
-LIBS:contrib
-LIBS:valves
-LIBS:usb_power_switcher-cache
-EELAYER 25 0
+EESchema Schematic File Version 4
+EELAYER 30 0
 EELAYER END
 $Descr A4 11693 8268
@@
 $EndDescr
 $Comp
-L USB_A J1
+L usb_power_switcher-rescue:USB_A J1
 U 1 1 5A876DAA
 P 3200 3450
@@
 $EndComp
 $Comp
-L USB_A J3
+L usb_power_switcher-rescue:USB_A J3
 U 1 1 5A876E02
 P 4850 3450
@@
 $EndComp
 $Comp
-L GND #PWR01
+L usb_power_switcher-rescue:GND #PWR01
 U 1 1 5A876E3C
 P 3200 3850
@@
 $EndComp
 $Comp
-L GND #PWR02
+L usb_power_switcher-rescue:GND #PWR02
 U 1 1 5A876E54
 P 4850 3850
@@
 $EndComp
 $Comp
-L Earth #PWR03
+L usb_power_switcher-rescue:Earth #PWR03
 U 1 1 5A876E85
 P 3100 3850
@@
 $EndComp
 $Comp
-L Earth #PWR04
+L usb_power_switcher-rescue:Earth #PWR04
 U 1 1 5A876E9D
 P 4750 3850
@@
 D-
 $Comp
-L +5V #PWR05
+L usb_power_switcher-rescue:+5V #PWR05
 U 1 1 5A876ED4
 P 3550 3200
@@
 $EndComp
 $Comp
-L +5VD #PWR06
+L usb_power_switcher-rescue:+5VD #PWR06
 U 1 1 5A876EEC
 P 5200 3200
@@
 $EndComp
 $Comp
-L R_Small R2
+L usb_power_switcher-rescue:R_Small R2
 U 1 1 5A876F56
 P 3350 4650
@@
 $EndComp
 $Comp
-L Conn_01x04 J2
+L usb_power_switcher-rescue:Conn_01x04 J2
 U 1 1 5A876FD8
 P 4150 3050
@@
 $EndComp
 $Comp
-L +5VD #PWR07
+L usb_power_switcher-rescue:+5VD #PWR07
 U 1 1 5A877023
 P 4500 3200
@@
 $EndComp
 $Comp
-L +5V #PWR08
+L usb_power_switcher-rescue:+5V #PWR08
 U 1 1 5A87703A
 P 3900 3200
@@
 $EndComp
 $Comp
-L GND #PWR09
+L usb_power_switcher-rescue:GND #PWR09
 U 1 1 5A8770B4
 P 4250 3300
@@
 CTRL
 $Comp
-L R_Small R3
+L usb_power_switcher-rescue:R_Small R3
 U 1 1 5A87717B
 P 3350 4950
@@
 $EndComp
 $Comp
-L GND #PWR010
+L usb_power_switcher-rescue:GND #PWR010
 U 1 1 5A8771D6
 P 3350 5050
@@
 $EndComp
 $Comp
-L +5V #PWR011
+L usb_power_switcher-rescue:+5V #PWR011
 U 1 1 5A8771F5
 P 3350 4550
@@
 $EndComp
 $Comp
-L GS2 J4
+L usb_power_switcher-rescue:GS2 J4
 U 1 1 5A87731C
 P 5350 3450
@@
 $EndComp
 $Comp
-L GS2 J5
+L usb_power_switcher-rescue:GS2 J5
 U 1 1 5A877409
 P 5350 3550
@@
 $EndComp
 $Comp
-L R_Small R1
+L usb_power_switcher-rescue:R_Small R1
 U 1 1 5A877708
 P 3500 4800
@@
 $EndComp
 $Comp
-L GND #PWR012
+L usb_power_switcher-rescue:GND #PWR012
 U 1 1 5A877A5A
 P 3900 5000
@@
 $EndComp
 $Comp
-L Q_PMOS_GSD Q2
+L usb_power_switcher-rescue:Q_PMOS_GSD Q2
 U 1 1 5A877AC8
 P 4400 4700
@@
 $EndComp
 $Comp
-L +5VD #PWR013
+L usb_power_switcher-rescue:+5VD #PWR013
 U 1 1 5A877B9D
 P 4500 4500
@@
 $EndComp
 $Comp
-L +5V #PWR014
+L usb_power_switcher-rescue:+5V #PWR014
 U 1 1 5A877BC6
 P 4500 5000
@@
 $EndComp
 $Comp
-L R_Small R4
+L usb_power_switcher-rescue:R_Small R4
 U 1 1 5A877CB3
 P 4150 4800
@@
 $EndComp
 $Comp
-L LED D1
+L usb_power_switcher-rescue:LED D1
 U 1 1 5A878320
 P 2750 3500
@@
 $EndComp
 $Comp
-L +5V #PWR015
+L usb_power_switcher-rescue:+5V #PWR015
 U 1 1 5A8783A1
 P 2750 3350
@@
 $EndComp
 $Comp
-L R_Small R5
+L usb_power_switcher-rescue:R_Small R5
 U 1 1 5A8783FF
 P 2750 3750
@@
 $EndComp
 $Comp
-L GND #PWR016
+L usb_power_switcher-rescue:GND #PWR016
 U 1 1 5A87844C
 P 2750 3850
@@
 $EndComp
 $Comp
-L LED D2
+L usb_power_switcher-rescue:LED D2
 U 1 1 5A8784DE
 P 6000 3400
@@
 $EndComp
 $Comp
-L R_Small R6
+L usb_power_switcher-rescue:R_Small R6
 U 1 1 5A8784EA
 P 6000 3650
@@
 $EndComp
 $Comp
-L GND #PWR017
+L usb_power_switcher-rescue:GND #PWR017
 U 1 1 5A8784F0
 P 6000 3750
@@
 Connection ~ 5150 3450
 Connection ~ 5150 3550
-Connection ~ 5550 3550
-Connection ~ 5550 3450
 Wire Wire Line
 	4100 3400 4150 3400
@@
 	3900 4600 3900 4550
 Wire Wire Line
-	3900 4550 4200 4550
-Wire Wire Line
-	4500 4900 4500 5000
+	3900 4550 4150 4550
+Wire Wire Line
+	4500 4900 4500 4950
 Wire Wire Line
 	4500 4950 4150 4950
@@
 Connection ~ 4150 4550
 $Comp
-L +5VD #PWR018
+L usb_power_switcher-rescue:+5VD #PWR018
 U 1 1 5A878526
 P 6000 3250
@@
 $EndComp
 $Comp
-L LED D3
+L usb_power_switcher-rescue:LED D3
 U 1 1 5A878A72
 P 2750 5000
@@
 $EndComp
 $Comp
-L R_Small R7
+L usb_power_switcher-rescue:R_Small R7
 U 1 1 5A878A78
 P 2750 5250
@@
 $EndComp
 $Comp
-L GND #PWR019
+L usb_power_switcher-rescue:GND #PWR019
 U 1 1 5A878A7E
 P 2750 5350
@@
 	2750 4800 2750 4850
 $Comp
-L USB_OTG J6
+L usb_power_switcher-rescue:USB_OTG J6
 U 1 1 5AC0D2EF
 P 3200 2200
@@
 D-
 $Comp
-L +5V #PWR020
+L usb_power_switcher-rescue:+5V #PWR020
 U 1 1 5AC0D3EE
 P 3550 1950
@@
 	3550 2000 3550 1950
 $Comp
-L GND #PWR021
+L usb_power_switcher-rescue:GND #PWR021
 U 1 1 5AC0D513
 P 3200 2600
@@
 $EndComp
 $Comp
-L Earth #PWR022
+L usb_power_switcher-rescue:Earth #PWR022
 U 1 1 5AC0D554
 P 3100 2600
@@
 NoConn ~ 3500 2400
 Wire Wire Line
-	3200 4800 3400 4800
-Wire Wire Line
-	3350 4750 3350 4850
+	3200 4800 3350 4800
+Wire Wire Line
+	3350 4750 3350 4800
 Connection ~ 3350 4800
 $Comp
-L Q_NPN_BEC Q1
+L usb_power_switcher-rescue:Q_NPN_BEC Q1
 U 1 1 5BCD062D
 P 3800 4800
@@
 	1    0    0    -1
 $EndComp
+Wire Wire Line
+	4500 4950 4500 5000
+Wire Wire Line
+	4150 4550 4200 4550
+Wire Wire Line
+	3350 4800 3400 4800
+Wire Wire Line
+	3350 4800 3350 4850
 $EndSCHEMATC
