File: Power stuff/simple_fet_powerpath/simple_fet_powerpath.sch (KiCad schematic (older format))
At the start: 7 parts, among them Q1 IRLML6401

Commit message: Reloading the simple FET power path project files
Parts:
- D1: symbol D_Schottky_Small -> simple_fet_powerpath-rescue:D_Schottky_Small
- Q1: symbol Q_PMOS_GSD -> simple_fet_powerpath-rescue:Q_PMOS_GSD
- R1: symbol R_Small -> simple_fet_powerpath-rescue:R_Small
- W1, W2, W3, W4: symbol TEST_1P -> simple_fet_powerpath-rescue:TEST_1P
Changed lines of the file:
@@
-EESchema Schematic File Version 2
-LIBS:power
-LIBS:device
-LIBS:transistors
-LIBS:conn
-LIBS:linear
-LIBS:regul
-LIBS:74xx
-LIBS:cmos4000
-LIBS:adc-dac
-LIBS:memory
-LIBS:xilinx
-LIBS:microcontrollers
-LIBS:dsp
-LIBS:microchip
-LIBS:analog_switches
-LIBS:motorola
-LIBS:texas
-LIBS:intel
-LIBS:audio
-LIBS:interface
-LIBS:digital-audio
-LIBS:philips
-LIBS:display
-LIBS:cypress
-LIBS:siliconi
-LIBS:opto
-LIBS:atmel
-LIBS:contrib
-LIBS:valves
-EELAYER 25 0
+EESchema Schematic File Version 4
+EELAYER 30 0
 EELAYER END
 $Descr A4 11693 8268
@@
 $EndDescr
 $Comp
-L D_Schottky_Small D1
+L simple_fet_powerpath-rescue:D_Schottky_Small D1
 U 1 1 590E9A9A
 P 5000 4150
@@
 $EndComp
 $Comp
-L R_Small R1
+L simple_fet_powerpath-rescue:R_Small R1
 U 1 1 590E9B01
 P 4650 4350
@@
 $EndComp
 $Comp
-L TEST_1P W3
+L simple_fet_powerpath-rescue:TEST_1P W3
 U 1 1 590E9B46
 P 4550 4350
@@
 $EndComp
 $Comp
-L TEST_1P W4
+L simple_fet_powerpath-rescue:TEST_1P W4
 U 1 1 590E9C5C
 P 5200 3850
@@
 $EndComp
 $Comp
-L TEST_1P W2
+L simple_fet_powerpath-rescue:TEST_1P W2
 U 1 1 590E9CA1
 P 4550 4150
@@
 $EndComp
 $Comp
-L TEST_1P W1
+L simple_fet_powerpath-rescue:TEST_1P W1
 U 1 1 590E9D0F
 P 4550 3850
@@
 $EndComp
 $Comp
-L Q_PMOS_GSD Q1
+L simple_fet_powerpath-rescue:Q_PMOS_GSD Q1
 U 1 1 590E9D9C
 P 4800 3950
@@
 $EndComp
 Wire Wire Line
-	4550 4150 4900 4150
+	4550 4150 4800 4150
 Connection ~ 4800 4150
 Wire Wire Line
@@
 	4550 3850 4600 3850
 Wire Wire Line
-	5000 3850 5200 3850
+	5000 3850 5150 3850
 Wire Wire Line
 	5100 4150 5150 4150
@@
 	5150 4150 5150 3850
 Connection ~ 5150 3850
+Wire Wire Line
+	4800 4150 4900 4150
+Wire Wire Line
+	5150 3850 5200 3850
 $EndSCHEMATC
