File: ESP8266/protoesp/protoesp.sch (KiCad schematic (older format))
At the start: 25 parts

Commit message: ProtoESP schematic v2. Will be moved into the ESP32 directory next.
Parts:
- added C? (x2): 100nF, symbol Device:C_Small
- added C? (x3): 1uF, symbol Device:C_Small
- added D?: LED_RGBA, symbol Device:LED_RGBA
- added D? (x8): LED, symbol Device:LED_Small
- added D?: SS14, symbol Device:D_Schottky_Small
- added D?: LED_CHG, symbol Device:LED_Small
- added J?: RGB_CONN, symbol Connector_Generic:Conn_01x04
- added J?, JP? (x2): 0R, symbol Device:R_Small
- added J?: LDR_CONN, symbol Connector_Generic:Conn_01x03
- added J?: USB_CURSED, symbol Connector:USB_A
- added J?: CH_PROG, symbol Connector_Generic:Conn_01x02
- added J?: CH_SPI, symbol Connector_Generic:Conn_01x06
- added J?: CH_I2C, symbol Connector_Generic:Conn_01x05
- added J?: SPI, symbol Connector_Generic:Conn_01x06
- added J?: BATT, symbol Connector_Generic:Conn_01x02
- added JP?: F, symbol Device:R_Small
- added Q?: CJ2305, symbol Device:Q_PMOS_GSD
- added R? (x2): 4K7, symbol Device:R_Small
- added R?: RGB_R_B, symbol Device:R_Small
- added R?: RGB_R_G, symbol Device:R_Small
- added R?: RGB_R_R, symbol Device:R_Small
- added R? (x3): 1K8, symbol Device:R_Small
- added RN? (x2): R_Pack04, symbol Device:R_Pack04
- added U?: CH341, symbol ch341:CH341
- added U?: LTH7R, symbol LTH7R:LTH7R
Connections:
- net labels added: +5V, +BATT, CHG_VIN, CH_ACT, CH_CLK, CH_CS, CH_MISO, CH_MOSI, CH_RXD, CH_SCL, CH_SDA, CH_TXD, CH_VCC, D+, D-, E_SCL, E_SDA, LED_VCC
- wire segments 27 -> 132
- no-connect marks 6 -> 13
Other:
- note added: "CH341 USB-UART with I2C/SPI"
- note added: "CH341 board headers"
- note added: "Extra connectors"
- note added: "Powerpath and\nbattery charging"
- note removed: "Connectors"
- moved on the sheet: C?, J?, R?, U?

Commit message: ProtoESP schematic day 3
Parts:
- removed R?: 4K7, symbol Device:R_Small
- removed U?: ESP-12E, RF_Module:ESP-12E, symbol RF_Module:ESP-12E
- added C? (x2): 18pF, symbol Device:C_Small
- added C? (x3): 100nF, symbol Device:C_Small
- added D?: 1N4148, symbol Device:D_Small
- added JP? (x3): 0R, symbol Device:R_Small
- added NT? (x7): Net-Tie_2, symbol Device:Net-Tie_2
- added P?: PROTO_SPACE, symbol proto_space:PROTO_SPACE
- added Q?: BC817, symbol Device:Q_NPN_BEC
- added R? (x3): 1K8, symbol Device:R_Small
- added TP?: +, symbol Connector:TestPoint
- added TP?: -, symbol Connector:TestPoint
- added U?: AP1117-33, Package_TO_SOT_SMD:SOT-223-3_TabPin2, symbol Regulator_Linear:AP1117-33
- added U?: ESP32-WROOM-32, RF_Module:ESP32-WROOM-32, symbol esp32_physlayout:ESP32-WROOM-32
- added Y?: 12MHz, symbol Device:Crystal
- J?: value I2C -> E_I2C
- J?: value SPI -> E_SPI
Connections:
- net labels added: 595_CLK, 595_CLK_J, 595_DAT, 595_DAT_J, 595_LAT, 595_LAT_J, CH_GP0, CH_RST, DRIVER, E_CS, E_EN, E_INT, E_MISO, E_MOSI, E_RXD, E_SCK, E_TXD, LED_ESP, LED_GREEN, LED_RED, POT
- net labels removed: CLK_595, DAT_595, EEN, LAT_595, SCL, SDA, ~ERST
- wire segments 132 -> 171
- no-connect marks 13 -> 20
Other:
- note added: "CH341 board headers for SPI/I2C programming"
- note added: "ESP32 module"
- note added: "ESP32-CH341\ninterconnect"
- note added: "Extra 1117\nfor standalone\nCH341 use"
- note added: "ProtoESP schematic\nv1, by CRImier\n"
- note added: "Speaker/vibromotor\ndriver"
- note removed: "CH341 board headers"
- note removed: "ESP8266 in ESP12 module form"
- moved on the sheet: C?, D?, J?, JP?, Q?, R?, RN?, SW?, U?

Commit message: ProtoESP schematic and PCB, day 4
Parts:
- removed NT?: Net-Tie_2, symbol Device:Net-Tie_2
- removed R?: 0R, symbol Device:R_Small
- added CN36: DRV_CONN, Connector_PinHeader_2.54mm:PinHeader_1x03_P2.54mm_Vertical, symbol Connector_Generic:Conn_01x03
- added J1: 0R, Resistor_SMD:R_0603_1608Metric, symbol Device:R_Small
- added R12, R13, R14, R15: 47K, Resistor_SMD:R_0603_1608Metric, symbol Device:R_Small
- C1, C2: renamed from C?; footprint (none) -> Capacitor_SMD:C_0603_1608Metric
- C10, C11, C3, C4, C5, C6, C7, C8, C9: renamed from C?; footprint (none) -> Capacitor_SMD:C_0805_2012Metric
- CN1, CN2: renamed from J?; footprint (none) -> Connector_PinHeader_2.54mm:PinHeader_1x08_P2.54mm_Vertical
- CN11, CN34: renamed from J?; footprint (none) -> Connector_PinSocket_2.54mm:PinSocket_1x06_P2.54mm_Horizontal
- CN12, CN35: renamed from J?; footprint (none) -> Connector_PinSocket_2.54mm:PinSocket_1x05_P2.54mm_Horizontal
- CN13, CN3: renamed from J?; footprint (none) -> Connector_PinHeader_2.54mm:PinHeader_1x07_P2.54mm_Vertical
- CN14, CN20: renamed from J?; footprint (none) -> Connector_PinSocket_2.54mm:PinSocket_1x02_P2.54mm_Vertical
- CN30: renamed from J?; footprint (none) -> Connector_PinHeader_2.54mm:PinHeader_1x02_P2.54mm_Vertical
- CN31: renamed from J?; footprint (none) -> Connector_PinHeader_2.54mm:PinHeader_1x03_P2.54mm_Vertical
- CN32: renamed from J?; footprint (none) -> Connector_PinHeader_2.54mm:PinHeader_1x04_P2.54mm_Vertical
- CN33: renamed from J?; footprint (none) -> Connector_PinHeader_2.54mm:PinHeader_1x05_P2.54mm_Vertical
- CN47: renamed from J?; footprint (none) -> Connector_PinSocket_2.54mm:PinSocket_1x10_P2.54mm_Vertical
- D1: renamed from D?; footprint (none) -> Diode_SMD:D_SOD-123
- D10, D11, D2, D4, D5, D6, D7, D8, D9: renamed from D?; footprint (none) -> LED_SMD:LED_0805_2012Metric
- D12: renamed from D?; footprint (none) -> LED_SMD:LED_RGB_1210
- D3: renamed from D?; footprint (none) -> Diode_SMD:D_SMA
- J11, J17, J19, J22, J7, J8, J9: renamed from J?; footprint (none) -> Resistor_SMD:R_0603_1608Metric
- JP1, JP2, JP3, JP4, JP5, JP6: renamed from JP?; footprint (none) -> Resistor_SMD:R_0805_2012Metric
- NT1, NT2, NT3, NT4, NT6, NT7: renamed from NT?; footprint (none) -> NetTie:NetTie-2_SMD_Pad0.5mm
- Q1, Q2: renamed from Q?; footprint (none) -> Package_TO_SOT_SMD:SOT-23
- R1, R10, R11, R16, R19, R2, R3, R4, R5, R6, R7, R8, R9: renamed from R?; footprint (none) -> Resistor_SMD:R_0603_1608Metric
- RN1, RN2: renamed from RN?; footprint (none) -> Resistor_SMD:R_Array_Concave_4x0603
- SW1, SW2: renamed from SW?; footprint (none) -> Button_Switch_SMD:SW_SPST_SKQG_WithStem
- TP1, TP2: renamed from TP?; footprint (none) -> TestPoint:TestPoint_Pad_2.0x2.0mm
- U1: renamed from U?; footprint (none) -> Package_SO:SOIC-28W_7.5x18.7mm_P1.27mm
- U3: renamed from U?; footprint (none) -> Package_TO_SOT_SMD:SOT-23-5
- U4: renamed from U?; footprint (none) -> Package_SO:SOP-16_4.55x10.3mm_P1.27mm
- Y1: renamed from Y?; footprint (none) -> Crystal:Crystal_HC49-U_Vertical
- gave numbers to parts that had none: 6
Connections:
- net RXD is gone; now on net E_RXD: CN2.2 (Pin_2)
- net TXD is gone; now on net E_TXD: CN2.1 (Pin_1)
- net +5V: now also CN13.5 (Pin_5), R12.2
- net +BATT: now also R15.2
- net +VSW: now also CN36.1 (Pin_1); no longer CN13.5 (Pin_5)
- net 595_CLK: now also U6.13 (IO14)
- net 595_DAT: now also U6.16 (IO13)
- net 595_LAT: now also U6.23 (IO15)
- net BUTTON: no longer CN2.5 (Pin_5)
- net DRIVER: now also J1.2
- net E_CS: now also CN1.7 (Pin_7), U6.28 (IO17)
- net E_INT: now also CN2.5 (Pin_5), U6.27 (IO16)
- net E_MISO: now also CN1.5 (Pin_5), U6.31 (IO19)
- net E_MOSI: now also CN1.4 (Pin_4), U6.37 (IO23)
- net E_SCK: now also CN1.6 (Pin_6), U6.30 (IO18)
- net E_SCL: no longer CN2.3 (Pin_3)
- net E_SDA: no longer CN2.4 (Pin_4)
- net GND: now also CN36.3 (Pin_3), R13.2, R14.2
- net LED_BLUE: now also U6.12 (IO27)
- net LED_GREEN: now also U6.11 (IO26)
- net LED_RED: now also U6.10 (IO25)
- net IO12: now reaches CN1.3 (Pin_3)
- net IO12: now also U6.14 (IO12)
- net at SW2.1: now also CN30.1 (Pin_1), J22.2
- net IO4: now reaches U6.26 (IO4)
- net IO4: now also CN2.4 (Pin_4)
- net IO5: now reaches U6.29 (IO5)
- net IO5: now also CN2.3 (Pin_3)
- net VUSB: now reaches U6.8 (IO32)
- net VUSB: now also R14.1, R15.1
- net VBAT: now reaches U6.9 (IO33)
- net VBAT: now also R12.1, R13.1
- new net: CN36.2 (Pin_2), J1.1
Other:
- moved on the sheet: C10, CN1, SW1

Commit message: ProtoESP work day 5, oh wait, actually, 6!
Parts:
- removed NT4: Net-Tie_2, NetTie:NetTie-2_SMD_Pad0.5mm, symbol Device:Net-Tie_2
- added C12: 100nF, Capacitor_SMD:C_0805_2012Metric, symbol Device:C_Small
- added D10: LED_5V, LED_SMD:LED_0805_2012Metric, symbol Device:LED_Small
- added D13: LED_3V3, LED_SMD:LED_0805_2012Metric, symbol Device:LED_Small
- added D14: LED_ESP, LED_SMD:LED_0805_2012Metric, symbol Device:LED_Small
- added R18, R20, R21: 1K8, Resistor_SMD:R_0603_1608Metric, symbol Device:R_Small
- CN10: footprint (none) -> protoesp:USB_Combined
- renumbered D4 to D0, D8 to D1, D1 to D11, D5 to D2, D9 to D3, D6 to D4, D10 to D5, D7 to D6, D11 to D7, D3 to D8, D2 to D9
Connections:
- net +3V3: now also CN31.1 (Pin_1), R16.2, D13.2 (A), D14.2 (A)
- net +5V: now also D10.2 (A)
- net +VSW: no longer CN36.1 (Pin_1)
- net DRIVER: no longer R1.1
- net GND: now also C12.2, R18.1, R20.1
- net LED_ESP: now also R21.1
- net LIGHT: no longer CN31.2 (Pin_2)
- net VBAT: now also R14.1, R15.1; no longer R12.1, R13.1
- net VUSB: now also R12.1, R13.1; no longer R14.1, R15.1
- net LIGHT_J: now reaches J19.2, R16.1, R17.1
- net LIGHT_J: now also CN31.2 (Pin_2), C12.1
- net at RN1.5 (R4.2): now also D3.1 (K); no longer D0.1 (K)
- net at RN1.6 (R3.2): now also D2.1 (K); no longer D1.1 (K)
- net at RN1.7 (R2.2): now also D1.1 (K); no longer D2.1 (K)
- net at RN1.8 (R1.2): now also D0.1 (K); no longer D3.1 (K)
- net at RN2.5 (R4.2): now also D7.1 (K); no longer D4.1 (K)
- net at RN2.6 (R3.2): now also D6.1 (K); no longer D5.1 (K)
- net at RN2.7 (R2.2): now also D5.1 (K); no longer D6.1 (K)
- net at RN2.8 (R1.2): now also D4.1 (K); no longer D7.1 (K)
- net BUTTON_J: now reaches CN30.1 (Pin_1), J22.2, SW2.1
- net at CN36.2 (Pin_2), J1.1: now also R1.1
- net at D11.1 (K), JP2.2, TP1.1: now also CN36.1 (Pin_1)
- new net: D14.1 (K), R21.2
- new net: D13.1 (K), R20.2
- new net: D10.1 (K), R18.2
- no-connect marks 20 -> 21
Other:
- moved on the sheet: CN36, J1, J19, JP2, SW1

Commit message: ProtoESP work day 7
Parts:
- removed CN20: BATT, Connector_PinSocket_2.54mm:PinSocket_1x02_P2.54mm_Vertical, symbol Connector_Generic:Conn_01x02
- added C13: 1uF, Capacitor_SMD:C_0805_2012Metric, symbol Device:C_Small
- added C14: 100nF, Capacitor_SMD:C_0805_2012Metric, symbol Device:C_Small
- added CN20: BATT, protoesp:JST_PH_S2B-PH-SM4-TB_02x2.00mm_Angled, symbol Connector_Generic_MountingPin:Conn_01x02_MountingPin
- added CN35: 595CHAIN_CONN, Connector_PinHeader_2.54mm:PinHeader_1x05_P2.54mm_Vertical, symbol Connector_Generic:Conn_01x05
- added JP7: 0R, Resistor_SMD:R_0805_2012Metric, symbol Device:R_Small
- added TP3, TP7, TP8: B+, TestPoint:TestPoint_Pad_2.0x2.0mm, symbol Connector:TestPoint
- added TP4: 5V, TestPoint:TestPoint_Pad_2.0x2.0mm, symbol Connector:TestPoint
- added TP5, TP9: GND, TestPoint:TestPoint_Pad_2.0x2.0mm, symbol Connector:TestPoint
- added TP6: VS, TestPoint:TestPoint_Pad_2.0x2.0mm, symbol Connector:TestPoint
- added U7: CH340G, Package_SO:SOIC-16_3.9x9.9mm_P1.27mm, symbol Interface_USB:CH340G
- P1: footprint (none) -> protoesp:PROTO_THT_SMD_FULL
- renumbered CN47 to CN34, CN35 to CN36, CN34 to CN37, CN36 to CN38
Connections:
- net +3V3: now also P1.e, C13.1, C14.1; no longer P1.c
- net +5V: now also TP4.1
- net +BATT: now also CN20.1 (Pin_1), TP3.1, TP8.1
- net +VSW: now also TP6.1
- net 595_CLK_J: now also CN35.3 (Pin_3)
- net 595_LAT_J: now also CN35.4 (Pin_4)
- net CH_RXD: now also U7.3 (RXD)
- net CH_TXD: now also U7.2 (TXD)
- net D+: now also U7.5 (UD+)
- net D-: now also U7.6 (UD-)
- net E_INT: now also P1.f
- net GND: now also P1.c, C13.2, C14.2, CN20.MP (MountPin), CN35.5 (Pin_5), JP7.2, TP5.1, TP9.1, U7.1 (GND); no longer P1.e
- net VCC_595: now also CN35.1 (Pin_1)
- net 5D0: now reaches P1.d0
- net 5D0: now also CN34.2 (Pin_2), D0.2 (A), U4.15 (QA)
- net 5D1: now reaches P1.d1
- net 5D1: now also CN34.3 (Pin_3), D1.2 (A), U4.1 (QB)
- net 5D2: now reaches P1.d2
- net 5D2: now also CN34.4 (Pin_4), D2.2 (A), U4.2 (QC)
- net 5D3: now reaches P1.d3
- net 5D3: now also CN34.5 (Pin_5), D3.2 (A), U4.3 (QD)
- net 5D4: now reaches P1.d4
- net 5D4: now also CN34.6 (Pin_6), D4.2 (A), U4.4 (QE)
- net 5D5: now reaches P1.d5
- net 5D5: now also CN34.7 (Pin_7), D5.2 (A), U4.5 (QF)
- net 5D6: now reaches P1.d6
- net 5D6: now also CN34.8 (Pin_8), D6.2 (A), U4.6 (QG)
- net 5D7: now reaches P1.d7
- net 5D7: now also CN34.9 (Pin_9), D7.2 (A), U4.7 (QH)
- net 595_DAT_O: now reaches U4.9 (QH')
- net 595_DAT_O: now also CN35.2 (Pin_2)
- new net -BATT: CN20.2 (Pin_2), JP7.1, TP7.1
Other:
- note added: "Protection\nfootprint"
- note added: "Testpoints for reusability"
- moved on the sheet: C11, C7, C8, CN33, CN34, D0, D1, D2, D3, D4, D5, D6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

Commit message: ProtoESP work day 8, part A
Parts:
- removed U7: CH340G, Package_SO:SOIC-16_3.9x9.9mm_P1.27mm, symbol Interface_USB:CH340G
- added C15, C16: 100nF, Capacitor_SMD:C_0805_2012Metric, symbol Device:C_Small
- added J2: 0R, Resistor_SMD:R_0603_1608Metric, symbol Device:R_Small
- added JP8: 0R, Resistor_SMD:R_0805_2012Metric, symbol Device:R_Small
- U1: footprint Package_SO:SOIC-28W_7.5x18.7mm_P1.27mm -> protoesp:SOIC-28W_SOIC16_CH34x_Combined
Connections:
- net +3V3: now also J2.2; no longer CN31.1 (Pin_1), R16.2
- net +5V: no longer R12.2
- net CHG_VIN: now also R12.2
- net CH_VCC: now also JP8.1
- net DRIVER: now also U6.9 (IO33)
- net GND: now also C15.2, C16.2
- net LIGHT: now also U6.5 (SENSOR_VN); no longer CN1.2 (Pin_2), U6.7 (IO35)
- net POT: now also CN1.2 (Pin_2), U6.4 (SENSOR_VP); no longer U6.6 (IO34)
- net VBAT: now also U6.7 (IO35), C16.1; no longer U6.9 (IO33)
- net VUSB: now also U6.6 (IO34), C15.1; no longer U6.8 (IO32)
- net CH_XI: now reaches C1.1, U1.13 (XI), Y1.1
- net CH_XO: now reaches C2.1, U1.14 (XO), Y1.2
- net CH_~RTS: now reaches U1.21 (~RTS~/D6/DIN2)
- net CH_V3: now reaches C5.1, U1.9 (V3)
- net CH_V3: now also JP8.2
- new net: CN31.1 (Pin_1), J2.1, R16.2
- no-connect marks 21 -> 19
Other:
- moved on the sheet: CN10, CN11, CN12, CN14, JP1

Commit message: Final changes - only small silk art things left before I'll order it, otherwise, this is orderable!
Parts:
- added C17, C18, C19: 100nF, Capacitor_SMD:C_0805_2012Metric, symbol Device:C_Small
- added CN4: EPINS_TOP_E, Connector_PinHeader_2.54mm:PinHeader_1x04_P2.54mm_Vertical, symbol Connector_Generic:Conn_01x04
- added CN5: EPINS_BOTTOM_E, Connector_PinHeader_2.54mm:PinHeader_1x04_P2.54mm_Vertical, symbol Connector_Generic:Conn_01x04
- added FID1, FID2, FID3, FID4: Fiducial, Fiducial:Fiducial_1mm_Mask2mm, symbol Mechanical:Fiducial
- added J?: DRV, symbol Connector:Screw_Terminal_01x02
- added Q3, Q4: BC817, Package_TO_SOT_SMD:SOT-23, symbol Device:Q_NPN_BEC
- added R22, R25, R26: 4K7, Resistor_SMD:R_0603_1608Metric, symbol Device:R_Small
- added R23, R24: 1K8, Resistor_SMD:R_0603_1608Metric, symbol Device:R_Small
- added SW3: GP0, Button_Switch_SMD:SW_SPST_SKQG_WithStem, symbol Switch:SW_Push
- SW1: value RST -> EN
- TP7: value B+ -> B-
Connections:
- net +3V3: now also P1.d, C18.1, R22.2, R23.2, R24.2; no longer P1.e
- net +5V: now also C17.1
- net +VSW: now also P1.a; no longer P1.b
- net 595_CLK: now also CN5.3 (Pin_3)
- net 595_DAT: now also CN5.4 (Pin_4)
- net 595_LAT: now also CN5.2 (Pin_2)
- net BUTTON: now also U6.14 (IO12), CN5.1 (Pin_1); no longer CN3.6 (Pin_6), NT6.2, U6.25 (IO0)
- net CH_GP0: now also Q4.3 (C)
- net CH_MOSI: now also Q4.2 (E), R25.1
- net CH_~RTS: now also CN12.4 (Pin_4), Q3.2 (E), R26.1
- net E_EN: now also C19.1
- net E_INT: now also P1.e; no longer P1.f
- net E_SCL: now also P1.f, R24.1
- net E_SDA: now also P1.g, R23.1
- net GND: now also P1.b, C17.2, C18.2, C19.2, CN4.1 (Pin_1), SW3.1; no longer P1.d
- net LED_BLUE: now also CN4.4 (Pin_4)
- net LED_GREEN: now also CN4.3 (Pin_3)
- net LED_RED: now also CN4.2 (Pin_2)
- net LIGHT: now also U6.4 (SENSOR_VP); no longer U6.5 (SENSOR_VN)
- net DRV+: now reaches CN38.1 (Pin_1), D11.1 (K), JP2.2, TP1.1
- net DRV+: now also J?.1 (Pin_1)
- net DRV-: now reaches D11.2 (A), Q1.3 (C), TP2.1
- net DRV-: now also J?.2 (Pin_2)
- net IO32: now reaches U6.8 (IO32)
- net IO32: now also CN1.3 (Pin_3)
- net CH_RST renamed CH_EN
- net CH_EN: now also Q3.3 (C)
- removed net IO12: CN1.3 (Pin_3), U6.14 (IO12)
- net POT renamed IO39
- net IO39: now also U6.5 (SENSOR_VN); no longer U6.4 (SENSOR_VP)
- new net: Q3.1 (B), R25.2
- new net: Q4.1 (B), R26.2
- new net E_GP0: CN3.6 (Pin_6), NT6.2, R22.1, SW3.2, U6.25 (IO0)
- no-connect marks 19 -> 18
Other:
- moved on the sheet: C1, C15, C16, C2, C5, CN1, CN10, CN11, CN12, CN2, CN38, D10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

Commit message: Latest updates - consider this v1.1 ;-P
Parts:
- added H1, H2, H3, H4: MountingHole, MountingHole:MountingHole_3.2mm_M3, symbol Mechanical:MountingHole
- gave numbers to parts that had none: 1
Other:
- moved on the sheet: FID1, FID2, FID3, FID4
Changed lines of the file:
@@
 L Mechanical:Fiducial FID1
 U 1 1 61E5ADDE
-P 2700 5050
-F 0 "FID1" H 2785 5096 50  0000 L CNN
-F 1 "Fiducial" H 2785 5005 50  0000 L CNN
-F 2 "Fiducial:Fiducial_1mm_Mask2mm" H 2700 5050 50  0001 C CNN
-F 3 "~" H 2700 5050 50  0001 C CNN
-	1    2700 5050
+P 2500 5050
+F 0 "FID1" H 2585 5096 50  0000 L CNN
+F 1 "Fiducial" H 2585 5005 50  0000 L CNN
+F 2 "Fiducial:Fiducial_1mm_Mask2mm" H 2500 5050 50  0001 C CNN
+F 3 "~" H 2500 5050 50  0001 C CNN
+	1    2500 5050
 	1    0    0    -1
 $EndComp
@@
 L Mechanical:Fiducial FID2
 U 1 1 61E5CD16
-P 2700 5300
-F 0 "FID2" H 2785 5346 50  0000 L CNN
-F 1 "Fiducial" H 2785 5255 50  0000 L CNN
-F 2 "Fiducial:Fiducial_1mm_Mask2mm" H 2700 5300 50  0001 C CNN
-F 3 "~" H 2700 5300 50  0001 C CNN
-	1    2700 5300
+P 2500 5300
+F 0 "FID2" H 2585 5346 50  0000 L CNN
+F 1 "Fiducial" H 2585 5255 50  0000 L CNN
+F 2 "Fiducial:Fiducial_1mm_Mask2mm" H 2500 5300 50  0001 C CNN
+F 3 "~" H 2500 5300 50  0001 C CNN
+	1    2500 5300
 	1    0    0    -1
 $EndComp
@@
 L Mechanical:Fiducial FID3
 U 1 1 61E5CE93
-P 3250 5050
-F 0 "FID3" H 3335 5096 50  0000 L CNN
-F 1 "Fiducial" H 3335 5005 50  0000 L CNN
-F 2 "Fiducial:Fiducial_1mm_Mask2mm" H 3250 5050 50  0001 C CNN
-F 3 "~" H 3250 5050 50  0001 C CNN
-	1    3250 5050
+P 3000 5050
+F 0 "FID3" H 3085 5096 50  0000 L CNN
+F 1 "Fiducial" H 3085 5005 50  0000 L CNN
+F 2 "Fiducial:Fiducial_1mm_Mask2mm" H 3000 5050 50  0001 C CNN
+F 3 "~" H 3000 5050 50  0001 C CNN
+	1    3000 5050
 	1    0    0    -1
 $EndComp
@@
 L Mechanical:Fiducial FID4
 U 1 1 61E5D16D
-P 3250 5300
-F 0 "FID4" H 3335 5346 50  0000 L CNN
-F 1 "Fiducial" H 3335 5255 50  0000 L CNN
-F 2 "Fiducial:Fiducial_1mm_Mask2mm" H 3250 5300 50  0001 C CNN
-F 3 "~" H 3250 5300 50  0001 C CNN
-	1    3250 5300
+P 3000 5300
+F 0 "FID4" H 3085 5346 50  0000 L CNN
+F 1 "Fiducial" H 3085 5255 50  0000 L CNN
+F 2 "Fiducial:Fiducial_1mm_Mask2mm" H 3000 5300 50  0001 C CNN
+F 3 "~" H 3000 5300 50  0001 C CNN
+	1    3000 5300
 	1    0    0    -1
 $EndComp
@@
 DRV-
 $Comp
-L Connector:Screw_Terminal_01x02 J?
+L Connector:Screw_Terminal_01x02 J3
 U 1 1 61E69980
 P 600 5050
-F 0 "J?" H 518 5267 50  0000 C CNN
+F 0 "J3" H 518 5267 50  0000 C CNN
 F 1 "DRV" H 518 5176 50  0000 C CNN
 F 2 "" H 600 5050 50  0001 C CNN
@@
 Text GLabel 800  5150 2    50   Input ~ 0
 DRV-
+$Comp
+L Mechanical:MountingHole H1
+U 1 1 61EBE968
+P 3600 4800
+F 0 "H1" H 3700 4846 50  0000 L CNN
+F 1 "MountingHole" H 3700 4755 50  0000 L CNN
+F 2 "MountingHole:MountingHole_3.2mm_M3" H 3600 4800 50  0001 C CNN
+F 3 "~" H 3600 4800 50  0001 C CNN
+	1    3600 4800
+	1    0    0    -1
+$EndComp
+$Comp
+L Mechanical:MountingHole H2
+U 1 1 61EC04C0
+P 3600 5000
+F 0 "H2" H 3700 5046 50  0000 L CNN
+F 1 "MountingHole" H 3700 4955 50  0000 L CNN
+F 2 "MountingHole:MountingHole_3.2mm_M3" H 3600 5000 50  0001 C CNN
+F 3 "~" H 3600 5000 50  0001 C CNN
+	1    3600 5000
+	1    0    0    -1
+$EndComp
+$Comp
+L Mechanical:MountingHole H3
+U 1 1 61EC0837
+P 3600 5200
+F 0 "H3" H 3700 5246 50  0000 L CNN
+F 1 "MountingHole" H 3700 5155 50  0000 L CNN
+F 2 "MountingHole:MountingHole_3.2mm_M3" H 3600 5200 50  0001 C CNN
+F 3 "~" H 3600 5200 50  0001 C CNN
+	1    3600 5200
+	1    0    0    -1
+$EndComp
+$Comp
+L Mechanical:MountingHole H4
+U 1 1 61EC0B3E
+P 3600 5400
+F 0 "H4" H 3700 5446 50  0000 L CNN
+F 1 "MountingHole" H 3700 5355 50  0000 L CNN
+F 2 "MountingHole:MountingHole_3.2mm_M3" H 3600 5400 50  0001 C CNN
+F 3 "~" H 3600 5400 50  0001 C CNN
+	1    3600 5400
+	1    0    0    -1
+$EndComp
 $EndSCHEMATC
