File: ESP8266/protoesp/protoesp.kicad_pcb (KiCad board)
At the start: 2 copper layers, 100 x 95 mm, 93 parts, among them CN1 EPINS_TOP, CN11 CH_SPI, CN12 CH_I2C, CN13 CH341_PROG, CN14 CH_PROG, CN2 EPINS_BOTTOM, CN20 BATT, CN3 ESP_PROG, CN30 BUTTON_CONN, CN31 LDR_CONN, CN32 RGB_CONN, CN33 595_CONN, CN34 E_SPI, CN35 E_I2C, CN36 DRV_CONN, CN47 595_OUTS, J1 0R, J11 0R, J17 0R, J19 0R, J22 0R, J7 0R, J8 0R, J9 0R, Q1 BC817, Q2 CJ2305, SW1 RST, SW2 BUTTON, U1 CH341, U2 AP1117-33, U3 LTH7R, U4 74HC595, U5 AP2112K-3.3, U6 ESP32-WROOM-32, Y1 12MHz

Commit message: ProtoESP work day 5, oh wait, actually, 6!
Parts:
- removed the D7 at (218.3, 125.3)
- removed NT4, NT5: Net-Tie_2, NetTie:NetTie-2_SMD_Pad0.5mm
- added C12: 100nF, Capacitor_SMD:C_0805_2012Metric, F.Cu at (99.8, 111.4)
- added CN10: USB_CURSED, protoesp:USB_Combined, F.Cu at (52.8, 66.5)
- added D10: LED_5V, LED_SMD:LED_0805_2012Metric, F.Cu at (68.9, 77.0)
- added D13: LED_3V3, LED_SMD:LED_0805_2012Metric, F.Cu at (119.3, 69.7)
- added D14: LED_ESP, LED_SMD:LED_0805_2012Metric, F.Cu at (125.8, 71.6)
- added D6: LED, LED_SMD:LED_0805_2012Metric, F.Cu at (69.8, 132.6)
- added R18: 1K8, Resistor_SMD:R_0603_1608Metric, F.Cu at (72.2, 77.0)
- added R20: 1K8, Resistor_SMD:R_0603_1608Metric, F.Cu at (116.0, 69.6)
- added R21: 1K8, Resistor_SMD:R_0603_1608Metric, F.Cu at (125.8, 74.8)
- added REF**: mouse_1power_2sig_7.5mm, protoesp:mouse_1power_2sig_7.5mm, F.Cu at (77.2, 105.0)
- added REF**: mouse_1power_2sig_7.5mm, protoesp:mouse_1power_2sig_7.5mm, F.Cu at (87.2, 74.8)
- added REF**: mouse_1power_2sig_7.5mm, protoesp:mouse_1power_2sig_7.5mm, F.Cu at (97.5, 102.2)
- added REF**: mouse_1power_2sig_7.5mm, protoesp:mouse_1power_2sig_7.5mm, F.Cu at (97.5, 105.2)
- added REF**: mouse_1power_2sig_7.5mm, protoesp:mouse_1power_2sig_7.5mm, F.Cu at (82.5, 105.2)
- added REF**: mouse_1power_2sig_7.5mm, protoesp:mouse_1power_2sig_7.5mm, F.Cu at (82.5, 102.2)
- added REF**: mouse_1power_2sig_7.5mm, protoesp:mouse_1power_2sig_7.5mm, F.Cu at (77.8, 102.5)
- added REF**: mouse_1power_2sig_7.5mm, protoesp:mouse_1power_2sig_7.5mm, F.Cu at (105.2, 62.5)
- added REF**: mouse_1power_2sig_7.5mm, protoesp:mouse_1power_2sig_7.5mm, F.Cu at (102.2, 62.5)
- added REF**: mouse_1power_2sig_7.5mm, protoesp:mouse_1power_2sig_7.5mm, F.Cu at (90.2, 62.5)
- added REF**: mouse_1power_2sig_7.5mm, protoesp:mouse_1power_2sig_7.5mm, F.Cu at (87.2, 62.5)
- added REF**: mouse_1power_2sig_7.5mm, protoesp:mouse_1power_2sig_7.5mm, F.Cu at (105.2, 74.8)
- added REF**: mouse_1power_2sig_7.5mm, protoesp:mouse_1power_2sig_7.5mm, F.Cu at (102.2, 74.8)
- added REF**: mouse_1power_2sig_7.5mm, protoesp:mouse_1power_2sig_7.5mm, F.Cu at (90.2, 74.8)
- NT1, NT2, NT3, NT6, NT7: moved to B.Cu
- moved C1 192.6 mm to (61.8, 76.2)
- moved R2 192.4 mm to (62.2, 55.6)
- moved D5 190.4 mm to (69.8, 130.0)
- moved JP1 189.2 mm to (62.2, 71.0), turned to 90 degrees
- moved Q1 189.1 mm to (59.4, 95.2), turned to 180 degrees
- moved D4 186.6 mm to (69.8, 127.4)
- moved C2 181.9 mm to (55.4, 76.0)
- moved JP5 171.6 mm to (79.0, 56.6)
- moved R11 171.5 mm to (82.4, 111.6), turned to 90 degrees
- moved C5 171.4 mm to (63.8, 65.8), turned to 90 degrees
- moved R4 170.6 mm to (62.8, 129.4), turned to 180 degrees
- moved D0 170.6 mm to (69.8, 117.4)
- moved C8 169.5 mm to (62.2, 120.0)
- moved R1 168.1 mm to (62.0, 92.4), turned to 180 degrees
- moved J8 163.1 mm to (74.2, 100.3), turned to 270 degrees
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- renumbered D4 to D0, D8 to D1, D1 to D11, D5 to D2, D9 to D3, D6 to D4, D10 to D5, D11 to D7, D3 to D8, D2 to D9
Connections:
- net Net-(CN30-Pad1) renamed /BUTTON_J
- CN31 pad 1: Net-(CN31-Pad1) -> +3V3
- CN31 pad 2: LIGHT -> /LIGHT_J
- CN36 pad 1: +VSW -> Net-(CN36-Pad1)
- D0 pad 1: Net-(D4-Pad1) -> Net-(D0-Pad1)
- D1 pad 1: Net-(D8-Pad1) -> Net-(D1-Pad1)
- D11 pad 1: Net-(D1-Pad1) -> Net-(CN36-Pad1)
- D2 pad 1: Net-(D5-Pad1) -> Net-(D2-Pad1)
- D3 pad 1: Net-(D9-Pad1) (its old number) -> Net-(D3-Pad1)
- D4 pad 1: Net-(D6-Pad1) -> Net-(D4-Pad1)
- D5 pad 1: Net-(D10-Pad1) -> Net-(D5-Pad1)
- D7 pad 1: Net-(D11-Pad1) -> Net-(D7-Pad1)
- J19 pad 2: Net-(J19-Pad2) -> /LIGHT_J
- JP2 pad 2: Net-(D1-Pad1) -> Net-(CN36-Pad1)
- R1 pad 1: DRIVER -> Net-(CN36-Pad2)
- R12 pad 1: VBAT -> VUSB
- R13 pad 1: VBAT -> VUSB
- R14 pad 1: VUSB -> VBAT
- R15 pad 1: VUSB -> VBAT
- R16 pad 1: Net-(J19-Pad2) -> /LIGHT_J
- R16 pad 2: Net-(CN31-Pad1) -> +3V3
- R17 pad 1: Net-(J19-Pad2) -> /LIGHT_J
- RN1 pad 5: Net-(D4-Pad1) -> Net-(D3-Pad1)
- RN1 pad 6: Net-(D8-Pad1) -> Net-(D2-Pad1)
- RN1 pad 7: Net-(D5-Pad1) -> Net-(D1-Pad1)
- RN1 pad 8: Net-(D9-Pad1) (its old number) -> Net-(D0-Pad1)
- RN2 pad 5: Net-(D6-Pad1) -> Net-(D7-Pad1)
- RN2 pad 6: Net-(D10-Pad1) -> Net-(D6-Pad1)
- RN2 pad 7: Net-(D7-Pad1) -> Net-(D5-Pad1)
- RN2 pad 8: Net-(D11-Pad1) -> Net-(D4-Pad1)
- TP1 pad 1: Net-(D1-Pad1) -> Net-(CN36-Pad1)
Routing:
- net VCC_595: track 0.00 -> 54.3 mm, vias 0 -> 2
- net +3V3: track 0.00 -> 48.3 mm, vias 0 -> 4
- net 595_CLK_J: track 0.00 -> 45.1 mm, vias 0 -> 2
- net 595_LAT_J: track 0.00 -> 40.4 mm, vias 0 -> 1
- net 595_DAT_J: track 0.00 -> 38.6 mm
- net +BATT: track 0.00 -> 30.5 mm
- net Net-(CN47-Pad9): track 0.00 -> 27.9 mm, vias 0 -> 1
- net Net-(CN47-Pad8): track 0.00 -> 27.4 mm, vias 0 -> 1
- net Net-(CN47-Pad2): track 0.00 -> 27.1 mm, vias 0 -> 1
- net Net-(CN47-Pad7): track 0.00 -> 26.9 mm, vias 0 -> 1
- net Net-(CN47-Pad3): track 0.00 -> 26.9 mm, vias 0 -> 1
- net Net-(CN47-Pad6): track 0.00 -> 26.4 mm, vias 0 -> 1
- net Net-(CN47-Pad5): track 0.00 -> 25.8 mm, vias 0 -> 1
- net Net-(CN47-Pad4): track 0.00 -> 25.8 mm, vias 0 -> 1
- net LED_VCC: track 0.00 -> 24.0 mm
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Other:
- board size 100 x 95 mm -> 97.5 x 97.5 mm
- board text added: "595 shift register"
- board text added: "Button"
- board text added: "Driver"
- board text added: "Light"
- board text added: "ProtoESP ^_^ v1"
- board text added: "Prototyping space"
- board text added: "RGB LED"
- board text added: "by CRImier (Arsenijs)"
- board text removed: "ProtoESP ^__^"

Commit message: Day 6 continuation - mousebites done
Parts:
- added REF**: mouse_1sig_4.5mm, protoesp:mouse_1sig_4.5mm, F.Cu at (105.1, 54.9)
- added REF**: mouse_1power_2sig_7.5mm, protoesp:mouse_1power_2sig_7.5mm, F.Cu at (134.3, 89.8)
- added REF**: mouse_1power_2sig_7.5mm, protoesp:mouse_1power_2sig_7.5mm, F.Cu at (107.6, 92.6)
- added REF**: mouse_1power_2sig_7.5mm, protoesp:mouse_1power_2sig_7.5mm, F.Cu at (107.5, 89.8)
- added REF**: mouse_1power_2sig_7.5mm, protoesp:mouse_1power_2sig_7.5mm, F.Cu at (134.2, 102.4)
- added REF**: mouse_1power_2sig_7.5mm, protoesp:mouse_1power_2sig_7.5mm, F.Cu at (134.2, 105.2)
- added REF**: mouse_1power_2sig_7.5mm, protoesp:mouse_1power_2sig_7.5mm, F.Cu at (139.7, 92.6)
- added REF**: mouse_1power_2sig_7.5mm, protoesp:mouse_1power_2sig_7.5mm, F.Cu at (139.7, 89.8)
- added REF**: mouse_1power_2sig_7.5mm, protoesp:mouse_1power_2sig_7.5mm, F.Cu at (139.7, 105.2)
- added REF**: mouse_1power_2sig_7.5mm, protoesp:mouse_1power_2sig_7.5mm, F.Cu at (139.7, 102.4)
- added REF**: mouse_2sig_3mm, protoesp:mouse_2mm, F.Cu at (75.2, 85.0)
- added REF**: mouse_1sig_4.5mm, protoesp:mouse_1sig_4.5mm, F.Cu at (102.4, 54.9)
- added REF**: mouse_2sig_3mm, protoesp:mouse_2mm, F.Cu at (75.2, 82.5)
- added REF**: mouse_2sig_3mm, protoesp:mouse_2mm, F.Cu at (95.3, 85.0)
- added REF**: mouse_2sig_3mm, protoesp:mouse_2mm, F.Cu at (95.3, 82.5)
- added REF**: mouse_2sig_3mm, protoesp:mouse_2mm, F.Cu at (50.3, 102.5)
- added REF**: mouse_2sig_3mm, protoesp:mouse_2mm, F.Cu at (50.3, 105.0)
- added REF**: mouse_2sig_3mm, protoesp:mouse_2mm, F.Cu at (50.3, 82.5)
- added REF**: mouse_2sig_3mm, protoesp:mouse_2mm, F.Cu at (50.3, 85.0)
- added REF**: mouse_2sig_3mm, protoesp:mouse_2mm, F.Cu at (115.5, 122.5)
- added REF**: mouse_2sig_3mm, protoesp:mouse_2mm, F.Cu at (115.5, 125.0)
- added REF**: mouse_2sig_3mm, protoesp:mouse_2mm, F.Cu at (80.5, 125.0)
- added REF**: mouse_1sig_4.5mm, protoesp:mouse_1sig_4.5mm, F.Cu at (90.1, 54.9)
- added REF**: mouse_2sig_3mm, protoesp:mouse_2mm, F.Cu at (80.5, 122.5)
- added REF**: mouse_2sig_3mm, protoesp:mouse_2mm, F.Cu at (100.2, 122.5)
- added REF**: mouse_2sig_3mm, protoesp:mouse_2mm, F.Cu at (100.2, 125.0)
- added REF**: mouse_2sig_3mm, protoesp:mouse_2sig_3mm, F.Cu at (114.8, 105.0)
- added REF**: mouse_2sig_3mm, protoesp:mouse_2sig_3mm, F.Cu at (114.8, 102.5)
- added REF**: mouse_1sig_4.5mm, protoesp:mouse_1sig_4.5mm, F.Cu at (87.4, 54.9)
- added REF**: mouse_2sig_3mm, protoesp:mouse_2sig_3mm, F.Cu at (67.5, 94.0)
- added REF**: mouse_2sig_3mm, protoesp:mouse_2sig_3mm, F.Cu at (70.0, 94.0)
- added REF**: mouse_1sig_7.5mm, protoesp:mouse_1sig_7.5mm, F.Cu at (77.4, 139.6)
- added REF**: mouse_1sig_7.5mm, protoesp:mouse_1sig_7.5mm, F.Cu at (80.2, 139.6)
- added REF**: mouse_1power_2sig_7.5mm, protoesp:mouse_1power_2sig_7.5mm, F.Cu at (134.3, 92.6)
- moved J1 0.60 mm to (72.4, 93.5)
- moved JP2 0.60 mm to (72.5, 91.5)
- moved J22 0.50 mm to (115.5, 101.0)
Routing:
- net /BUTTON_J: track 0.00 -> 16.7 mm
- net +BATT: track 30.5 -> 43.6 mm
- net Net-(CN36-Pad1): track 15.0 -> 22.1 mm
- net Net-(CN36-Pad2): track 3.08 -> 9.65 mm
- net LED_RED: track 5.50 -> 11.8 mm
- net LED_BLUE: track 6.05 -> 12.1 mm
- net LED_GREEN: track 5.76 -> 11.4 mm
- net Net-(C3-Pad1): track 0.00 -> 4.64 mm
- net LED_VCC: track 24.0 -> 24.3 mm, vias 0 -> 2
Other:
- outline, holes or cut-outs redrawn

Commit message: ProtoESP work day 7
Parts:
- removed CN47: 595_OUTS, Connector_PinSocket_2.54mm:PinSocket_1x10_P2.54mm_Vertical
- removed the REF** at (134.2, 102.4)
- removed the REF** at (134.2, 105.2)
- removed the REF** at (95.3, 85.0)
- removed the REF** at (95.3, 82.5)
- removed the REF** at (97.5, 102.2)
- removed the REF** at (97.5, 105.2)
- removed the REF** at (82.5, 105.2)
- removed the REF** at (82.5, 102.2)
- removed the REF** at (77.4, 139.6)
- removed the REF** at (80.2, 139.6)
- added C13: 1uF, Capacitor_SMD:C_0805_2012Metric, F.Cu at (145.9, 58.2)
- added C14: 100nF, Capacitor_SMD:C_0805_2012Metric, F.Cu at (145.7, 80.8)
- added CN34: 595_OUTS, Connector_PinSocket_2.54mm:PinSocket_1x10_P2.54mm_Vertical, F.Cu at (75.0, 111.0)
- added CN36: E_I2C, Connector_PinSocket_2.54mm:PinSocket_1x05_P2.54mm_Horizontal, F.Cu at (143.3, 137.5)
- added JP7: 0R, Resistor_SMD:R_0805_2012Metric, F.Cu at (93.8, 60.5)
- added P1: PROTO_SPACE, protoesp:PROTO_THT_SMD_FULL, F.Cu at (127.0, 127.0)
- added REF**: mouse_2sig_3mm, protoesp:mouse_2mm_1sig, F.Cu at (105.0, 88.8)
- added REF**: mouse_2sig_3mm, protoesp:mouse_single, F.Cu at (76.7, 139.7)
- added REF**: mouse_2sig_3mm, protoesp:mouse_single, F.Cu at (80.8, 139.7)
- added REF**: mouse_2sig_3mm, protoesp:mouse_single, F.Cu at (147.2, 106.0)
- added REF**: mouse_2sig_3mm, protoesp:mouse_single, F.Cu at (147.2, 89.0)
- added REF**: mouse_2sig_3mm, protoesp:mouse_single, F.Cu at (86.6, 50.4)
- added REF**: mouse_2sig_3mm, protoesp:mouse_single, F.Cu at (90.9, 50.4)
- added REF**: mouse_2sig_3mm, protoesp:mouse_single, F.Cu at (101.6, 50.4)
- added REF**: mouse_2sig_3mm, protoesp:mouse_single, F.Cu at (105.9, 50.4)
- added REF**: mouse_2sig_3mm, protoesp:mouse_single, F.Cu at (91.0, 82.3)
- added REF**: mouse_2sig_3mm, protoesp:mouse_single, F.Cu at (86.5, 82.3)
- added REF**: mouse_2sig_3mm, protoesp:mouse_2mm_1sig, F.Cu at (102.5, 88.8)
- added REF**: mouse_2sig_3mm, protoesp:mouse_single, F.Cu at (50.3, 81.7)
- added REF**: mouse_2sig_3mm, protoesp:mouse_single, F.Cu at (50.3, 85.8)
- added REF**: mouse_2sig_3mm, protoesp:mouse_single, F.Cu at (50.3, 101.7)
- added REF**: mouse_2sig_3mm, protoesp:mouse_single, F.Cu at (50.3, 105.8)
- added REF**: mouse_2sig_3mm, protoesp:mouse_single, F.Cu at (105.1, 83.5)
- added REF**: mouse_1power_2sig_7.5mm, protoesp:mouse_1power_2sig_7.5mm, F.Cu at (77.4, 125.7)
- added REF**: mouse_1power_2sig_7.5mm, protoesp:mouse_1power_2sig_7.5mm, F.Cu at (80.2, 125.7)
- added REF**: mouse_2sig_3mm, protoesp:mouse_2mm, F.Cu at (77.5, 139.7)
- added REF**: mouse_2sig_3mm, protoesp:mouse_2mm, F.Cu at (80.0, 139.7)
- added REF**: mouse_2sig_3mm, protoesp:mouse_2mm_1sig, F.Cu at (95.3, 85.0)
- added REF**: mouse_1power_2sig_7.5mm, protoesp:mouse_1power_2sig_7.5mm, F.Cu at (126.7, 102.3)
- added REF**: mouse_2sig_3mm, protoesp:mouse_2mm_1sig, F.Cu at (95.3, 82.5)
- added REF**: mouse_1power_2sig_7.5mm, protoesp:mouse_1power_2sig_7.5mm, F.Cu at (126.8, 105.2)
- added REF**: mouse_2sig_3mm, protoesp:mouse_2sig_3mm, F.Cu at (84.5, 102.5)
- added REF**: mouse_2sig_3mm, protoesp:mouse_2sig_3mm, F.Cu at (84.5, 105.0)
- added REF**: mouse_2sig_3mm, protoesp:mouse_2sig_3mm, F.Cu at (99.8, 102.5)
- added REF**: mouse_2sig_3mm, protoesp:mouse_2sig_3mm, F.Cu at (99.8, 105.0)
- added REF**: mouse_2sig_3mm, protoesp:mouse_single, F.Cu at (80.4, 121.7)
- added TP3: B+, TestPoint:TestPoint_Pad_2.0x2.0mm, F.Cu at (100.7, 73.3)
- added TP4: 5V, TestPoint:TestPoint_Pad_2.0x2.0mm, F.Cu at (92.0, 78.6)
- added TP5: GND, TestPoint:TestPoint_Pad_2.0x2.0mm, F.Cu at (92.6, 73.4)
- added TP6: VS, TestPoint:TestPoint_Pad_2.0x2.0mm, F.Cu at (100.6, 78.6)
- added TP7: B+, TestPoint:TestPoint_Pad_2.0x2.0mm, B.Cu at (94.6, 60.1)
- added TP8: B+, TestPoint:TestPoint_Pad_2.0x2.0mm, B.Cu at (98.4, 60.1)
- added TP9: GND, TestPoint:TestPoint_Pad_2.0x2.0mm, B.Cu at (91.5, 60.1)
- added U7: CH340G, Package_SO:SOIC-16_3.9x9.9mm_P1.27mm, F.Cu at (66.0, 66.5)
- CN20: footprint Connector_PinSocket_2.54mm:PinSocket_1x02_P2.54mm_Vertical -> protoesp:JST_PH_S2B-PH-SM4-TB_02x2.00mm_Angled
- CN35: value E_I2C -> 595CHAIN_CONN; footprint Connector_PinSocket_2.54mm:PinSocket_1x05_P2.54mm_Horizontal -> Connector_PinHeader_2.54mm:PinHeader_1x05_P2.54mm_Vertical
- moved CN35 76.6 mm to (65.0, 132.9), turned to 270 degrees
- moved JP3 22.0 mm to (140.8, 136.6)
- moved C3 20.8 mm to (140.1, 139.1), turned to 180 degrees
- moved C4 14.1 mm to (141.0, 110.0)
- moved CN37 13.1 mm to (143.3, 122.3)
- moved JP4 11.8 mm to (141.0, 113.4), turned to 90 degrees
- moved REF** 7.50 mm to (126.8, 92.5), turned to 0 degrees
- moved REF** 7.50 mm to (126.8, 89.8), turned to 0 degrees
- moved C5 6.54 mm to (61.2, 59.8)
- moved R12 6.45 mm to (107.2, 61.0)
- moved R13 6.45 mm to (107.2, 59.5)
- moved R14 6.45 mm to (107.2, 58.0)
- moved R15 6.45 mm to (107.2, 56.5)
- moved U2 6.09 mm to (71.8, 73.4), turned to 90 degrees
- moved C11 5.69 mm to (117.5, 67.6), turned to 0 degrees
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- renumbered CN34 to CN37, CN36 to CN38
Connections:
- net Net-(CN47-Pad2) renamed /5D0
- net Net-(CN47-Pad3) renamed /5D1
- net Net-(CN47-Pad4) renamed /5D2
- net Net-(CN47-Pad5) renamed /5D3
- net Net-(CN47-Pad6) renamed /5D4
- net Net-(CN47-Pad7) renamed /5D5
- net Net-(CN47-Pad8) renamed /5D6
- net Net-(CN47-Pad9) renamed /5D7
- CN20 pad 2: GND -> -BATT
- CN35 pad 1: Net-(C3-Pad1) -> VCC_595
- CN35 pad 2: E_SDA -> 595_DAT_O
- CN35 pad 3: E_SCL -> 595_CLK_J
- CN35 pad 4: E_INT -> 595_LAT_J
- U4 pad 9: Net-(U4-Pad9) -> 595_DAT_O
Routing:
- net +3V3: track 48.3 -> 301.9 mm, vias 4 -> 10
- net GND: track 8.92 -> 111.8 mm, vias 5 -> 23
- net 595_CLK: track 0.00 -> 100.3 mm, vias 0 -> 3
- net +VSW: track 14.3 -> 109.2 mm, vias 2 -> 8
- net LED_RED: track 11.8 -> 104.2 mm, vias 0 -> 3
- net 595_DAT: track 0.00 -> 91.0 mm, vias 0 -> 3
- net LED_GREEN: track 11.4 -> 100.6 mm, vias 0 -> 3
- net LED_BLUE: track 12.1 -> 99.4 mm, vias 0 -> 4
- net 595_LAT: track 0.00 -> 85.8 mm, vias 0 -> 4
- net E_INT: track 0.00 -> 79.3 mm, vias 0 -> 1
- net E_MOSI: track 0.00 -> 76.9 mm, vias 0 -> 3
- net E_MISO: track 0.00 -> 76.1 mm, vias 0 -> 3
- net E_SCL: track 0.00 -> 75.6 mm, vias 0 -> 1
- net E_SCK: track 0.00 -> 75.3 mm, vias 0 -> 2
- net E_CS: track 0.00 -> 75.1 mm, vias 0 -> 2
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- added copper zone on F.Cu, net +VSW
Other:
- board size 97.5 x 97.5 mm -> 97.5 x 90 mm
- board text added: "- +"
- board text added: "3.3V D0 D1 D2 D3 D4 D5 D6 D7 GND"
- board text added: "3.3V DAT CLK LAT GND"
- board text added: "3.3V DATO CLK LAT GND"
- board text added: "3.3V DAT_O CLK LAT GND"
- board text added: "GND D+ D- 5V"
- board text added: "Power"
- board text added: "Prototyping space! I trust you to do something cool with it ^__^"
- board text added: "VSW GND"
- board text added: "black"
- board text added: "minus"
- board text added: "plus"
- board text added: "red"
- board text removed: "Prototyping space"

Commit message: ProtoESP work day 8, part A
Parts:
- removed the REF** at (86.6, 50.4)
- removed the REF** at (90.9, 50.4)
- removed the REF** at (101.6, 50.4)
- removed the REF** at (105.9, 50.4)
- removed the REF** at (105.1, 54.9)
- removed the REF** at (102.4, 54.9)
- removed the REF** at (90.1, 54.9)
- removed the REF** at (87.4, 54.9)
- removed the REF** at (80.5, 125.0)
- removed the REF** at (80.5, 122.5)
- removed the REF** at (80.4, 121.7)
- removed U7: CH340G, Package_SO:SOIC-16_3.9x9.9mm_P1.27mm
- added C15: 100nF, Capacitor_SMD:C_0805_2012Metric, F.Cu at (109.6, 60.4)
- added C16: 100nF, Capacitor_SMD:C_0805_2012Metric, F.Cu at (109.6, 57.1)
- added J2: 0R, Resistor_SMD:R_0603_1608Metric, F.Cu at (98.2, 101.0)
- added JP8: 0R, Resistor_SMD:R_0805_2012Metric, F.Cu at (64.2, 61.6)
- added REF**: mouse_2sig_3mm, protoesp:mouse_single, F.Cu at (77.2, 105.8)
- added REF**: mouse_2sig_3mm, protoesp:mouse_2mm_1sig, F.Cu at (102.5, 50.4)
- added REF**: mouse_2sig_3mm, protoesp:mouse_single, F.Cu at (105.8, 50.4)
- added REF**: mouse_2sig_3mm, protoesp:mouse_single, F.Cu at (101.7, 50.4)
- added REF**: mouse_2sig_3mm, protoesp:mouse_single, F.Cu at (86.7, 50.4)
- added REF**: mouse_2sig_3mm, protoesp:mouse_single, F.Cu at (90.8, 50.4)
- added REF**: mouse_2sig_3mm, protoesp:mouse_2mm, F.Cu at (87.5, 50.4)
- added REF**: mouse_2sig_3mm, protoesp:mouse_2mm, F.Cu at (90.0, 50.4)
- added REF**: mouse_2sig_3mm, protoesp:mouse_2mm, F.Cu at (125.0, 116.0)
- added REF**: mouse_2sig_3mm, protoesp:mouse_2mm, F.Cu at (122.5, 116.0)
- added REF**: mouse_2sig_3mm, protoesp:mouse_2mm, F.Cu at (85.0, 125.0)
- added REF**: mouse_2sig_3mm, protoesp:mouse_3mm, F.Cu at (53.2, 60.5)
- added REF**: mouse_2sig_3mm, protoesp:mouse_2mm, F.Cu at (85.0, 122.5)
- added REF**: mouse_2sig_3mm, protoesp:mouse_3mm, F.Cu at (53.2, 64.2)
- added REF**: mouse_2sig_3mm, protoesp:mouse_3mm, F.Cu at (53.2, 68.0)
- added REF**: mouse_2sig_3mm, protoesp:mouse_3mm, F.Cu at (53.2, 71.8)
- added REF**: mouse_2sig_3mm, protoesp:mouse_3mm, F.Cu at (53.2, 75.5)
- added REF**: mouse_2sig_3mm, protoesp:mouse_3mm, F.Cu at (53.2, 76.5)
- added REF**: mouse_2sig_3mm, protoesp:mouse_3mm, F.Cu at (53.2, 56.5)
- added REF**: mouse_2sig_3mm, protoesp:mouse_2mm_1sig, F.Cu at (105.0, 50.4)
- U1: footprint Package_SO:SOIC-28W_7.5x18.7mm_P1.27mm -> protoesp:SOIC-28W_SOIC16_CH34x_Combined
- moved R2 17.4 mm to (79.6, 55.9)
- moved Y1 7.07 mm to (62.0, 77.2), turned to 180 degrees
- moved C2 5.76 mm to (58.2, 81.0)
- moved C1 4.88 mm to (61.3, 81.0), turned to 180 degrees
- moved C5 4.75 mm to (61.9, 64.5)
- moved R18 3.63 mm to (75.8, 77.5)
- moved D10 3.63 mm to (72.5, 77.4)
- moved U2 3.48 mm to (74.5, 75.6)
- moved CN14 1.45 mm to (82.5, 52.5), turned to 90 degrees
- moved U1 1.25 mm to (71.9, 65.6)
- moved D12 1.25 mm to (86.2, 115.0)
- moved JP5 1.14 mm to (79.7, 57.5)
- moved R17 0.63 mm to (103.0, 115.0)
- moved SW2 0.21 mm to (116.2, 115.0)
- moved JP1 0.07 mm to (60.9, 72.5), turned to 180 degrees
Connections:
- net Net-(C1-Pad1) renamed /CH_XI
- net Net-(C2-Pad1) renamed /CH_XO
- net Net-(C5-Pad1) renamed CH_V3
- net Net-(U1-Pad21) renamed CH_~RTS
- CN1 pad 2: LIGHT -> POT
- CN31 pad 1: +3V3 -> Net-(CN31-Pad1)
- R12 pad 2: +5V -> CHG_VIN
- R16 pad 2: +3V3 -> Net-(CN31-Pad1)
- U6 pad 4: Net-(U6-Pad4) -> POT
- U6 pad 5: Net-(U6-Pad5) -> LIGHT
- U6 pad 6: POT -> VUSB
- U6 pad 7: LIGHT -> VBAT
- U6 pad 8: VUSB -> Net-(U6-Pad8)
- U6 pad 9: VBAT -> DRIVER
Routing:
- net GND: track 111.8 -> 197.0 mm, vias 23 -> 118
- net DRIVER: track 44.2 -> 112.8 mm, vias 2 -> 3
- net CH_VCC: track 0.00 -> 52.7 mm
- net +5V: track 19.4 -> 59.1 mm, vias 2 -> 5
- net CH_CS: track 0.00 -> 35.6 mm, vias 0 -> 1
- net +3V3: track 301.9 -> 336.4 mm, vias 10 -> 8
- net CHG_VIN: track 10.2 -> 41.4 mm, vias 0 -> 3
- net CH_CLK: track 0.00 -> 30.0 mm, vias 0 -> 1
- net CH_MOSI: track 0.00 -> 28.8 mm, vias 0 -> 1
- net CH_TXD: track 12.0 -> 39.2 mm, vias 0 -> 3
- net CH_RXD: track 12.4 -> 39.3 mm, vias 0 -> 3
- net CH_MISO: track 0.00 -> 22.7 mm, vias 0 -> 1
- net /CH_XO: track 0.00 -> 22.5 mm
- net /CH_XI: track 0.00 -> 20.3 mm
- net +BATT: track 26.2 -> 46.5 mm, vias 0 -> 2
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- added copper zone on B.Cu, net (none)
- added copper zone on F.Cu, net (none)
- added copper zone on B.Cu, net GND
- added copper zone on F.Cu, net GND
Other:
- outline, holes or cut-outs redrawn
- board text added: "+ -"
- board text added: "+V S G"
- board text added: ","
- board text added: "3.3V RXD TXD GND VSW GP0 EN"
- board text added: "3.3V TXD RXD GND 5V GP0 EN"
- board text added: "5V"
- board text added: "B G"
- board text added: "B G R +V"
- board text added: "B+"
- board text added: "GND"
- board text added: "GND ACT CVCC CSDA CSCL NC GND CMOSI CMISO CCLK CCS CVCC GND"
- board text added: "GP0"
- board text added: "GP13 14 15"
- board text added: "GP27 26 25"
- board text added: "GP33"
- board text added: "GP35"
- board text added: "ProtoESP 595 PCB v1"
- board text added: "ProtoESP CH340/1 PCB v1"
- board text added: "ProtoESP Driver PCB v1"
- board text added: "ProtoESP RGB PCB v1"
- board text added: "ProtoESP button PCB v1"
- board text added: "ProtoESP light PCB v1"
- board text added: "ProtoESP power PCB v1"
- board text added: "VS"
- board text added: "VSW DRV GND"
- board text added: "bat tery in put"
- board text added: "d 0 1 2 3 4 5 6 7"
- board text added: "why do I even clock"
- board text added: "~~"
- board text removed: "VSW GND"
