File: ESP8266/protoesp/protoesp.kicad_sch (KiCad schematic)
At the start: 144 parts, among them CN1 EPINS_TOP, CN10 USB_CURSED, CN11 CH_SPI, CN12 CH_I2C, CN13 CH341_PROG, CN14 CH_PROG, CN2 EPINS_BOTTOM, CN20 BATT, CN3 ESP_PROG, CN30 BUTTON_CONN, CN31 LDR_CONN, CN32 RGB_CONN, CN33 595_CONN, CN34 595_OUTS, CN35 595CHAIN_CONN, CN36 E_I2C, CN37 E_SPI, CN38 DRV_CONN, CN39 DRV, CN4 EPINS_TOP_E, CN5 EPINS_BOTTOM_E, J1 0R, J11 0R, J17 0R, J19 0R, J2 0R, J22 0R, J7 0R, J8 0R, J9 0R, P1 PROTO_SPACE, Q1 BC817, Q2 CJ2305, Q3 BC817, Q4 BC817, SW1 EN, SW2 BUTTON, SW3 GP0, U1 CH341, U2 AP1117-33, U3 LTH7R, U4 74HC595, U5 AP2112K-3.3, U6 ESP32-WROOM-32, Y1 12MHz

Commit message: protoesp: idk what changes are there, kicad diffs are unreadable, so just consider this change-less update to Kicad7
Parts:
- added CN6: QWIIC, Connector_JST:JST_SH_BM04B-SRSS-TB_1x04-1MP_P1.00mm_Vertical, symbol Connector_Generic_MountingPin:Conn_01x04_MountingPin
Connections:
- net +3V3: now also CN6.2 (Pin_2)
- net E_SCL: now also CN6.4 (Pin_4)
- net E_SDA: now also CN6.3 (Pin_3)
- net GND: now also CN6.1 (Pin_1), CN6.MP (MountPin)
Other:
- note added: "QWIIC"
- moved on the sheet: CN32, D12, J17, R10, R11, R9
