File: Reverse-engineering/usbc_debug_finder/usbc_debug_finder.kicad_sch (KiCad schematic)
At the start: 22 parts, among them J1 USB_C_Plug

Commit message: usbc_debug_finder: v1 (new, actual to-be-ordered)
Parts:
- BT1: footprint Battery:Battery_Panasonic_CR1220-VCN_Vertical_CircularHoles -> usbc_debug_finder:BAT-TH_BS-05-A1BJ001
Changed lines of the file:
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@@
       (effects (font (size 1.27 1.27)) (justify right))
     )
-    (property "Footprint" "Battery:Battery_Panasonic_CR1220-VCN_Vertical_CircularHoles" (at 133.35 78.359 90)
+    (property "Footprint" "usbc_debug_finder:BAT-TH_BS-05-A1BJ001" (at 133.35 78.359 90)
       (effects (font (size 1.27 1.27)) hide)
     )
