File: Wearables/hapticbelt_driver/hapticbelt_driver.kicad_pcb (KiCad board)
At the start: 2 copper layers, 17 x 17 mm, 19 parts, among them J1 FPC1, J2 FPC2, J3 OUTB, J4 OUTG, J5 OUTR, J6 FPCB1, J7 FPCB2, Q1 Q_PMOS_GSD, Q2 Q_PMOS_GSD, Q3 Q_PMOS_GSD, U1 WS2818B

Commit message: hapticbelt_driver: actually manufactured v1 version, with seriously improved silk
Other:
- board text added: "trans rights"
Changed lines of the file:
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@@
     (effects (font (size 0.8 0.8) (thickness 0.1)) (justify left bottom mirror))
+  )
+  (gr_text "trans\nrights" (at 104.902 66.294 45) (layer "B.SilkS")
+    (effects (font (size 0.8 0.8) (thickness 0.12)) (justify bottom mirror))
   )
   (gr_text "Haptic belt driver\nby Arya, v1" (at 103.625 58.9) (layer "B.SilkS")
