File: Reverse-engineering/sony_vaio_p_re/vaio_re.kicad_sch (KiCad schematic)
At the start: 112 parts, among them IC1 SN75LVDS83B, J1 RPi_GPIO, J2 AXK750147G_VAIO-P, J3 AXK760347G_VAIO-P, J4 qwiic, J6 20374-R30E-31, U1 AP2112K-3.3, U10 LP8551TLX/NOPB, U2 PAM2306AYPAA, U3 SL2.1A, U4 RP2040, U5 W25Q128JVS, U6 RP2040, U7 W25Q128JVS, U8 FSUSB42MUX, U9 SY6280, Y1 12MHz, Y2 ABM8-272-T3, Y3 ABM8-272-T3

Commit message: sony_vaio_p_re: working away
Parts:
- removed U10: LP8551TLX/NOPB, lib:DSBGA-25_L2.5-W2.5-R5-C5-P0.50-BL, symbol LP8551:LP8551TLX_NOPB
- added J5: qwiic?, Connector_JST:JST_SH_SM04B-SRSS-TB_1x04-1MP_P1.00mm_Horizontal, symbol Connector_Generic_MountingPin:Conn_01x04_MountingPin
- added Q1, Q2: 2N7002, Package_TO_SOT_SMD:SOT-23, symbol Transistor_FET:2N7002
- added R32, R33, R40, R41: 27, Resistor_SMD:R_0402_1005Metric, symbol Device:R
- added R34, R35, R42, R43: 4.7K, Resistor_SMD:R_0402_1005Metric, symbol Device:R
- added R36, R37, R38, R39: Pu, Resistor_SMD:R_0402_1005Metric, symbol Device:R
- added U12, U13: 74HC595, Package_SO:SO-16_3.9x9.9mm_P1.27mm, symbol 74xx:74HC595
Connections:
- net +3V3: now also J5.2 (Pin_2), R36.1, R37.1, R38.1, R39.1; no longer J2.43 (+3VALW), J4.2 (Pin_2)
- net +3V3E: now also J2.43 (+3VALW), J4.2 (Pin_2), R35.1, R43.1, U12.16 (VCC), U13.16 (VCC)
- net EN_2V5: now also U13.2 (QC); no longer U6.37 (GPIO25)
- net EN_3V3: now also U13.4 (QE); no longer U6.36 (GPIO24)
- net GND: now also J5.1 (Pin_1), J5.MP (MountPin), Q1.2 (S), Q2.2 (S), R34.2, R42.2, U12.8 (GND), U13.8 (GND); no longer J2.33 (LED_RTN)
- net KB_BOOT: now also R41.2; no longer R11.1
- net KB_RX: now also J5.4 (Pin_4), R32.1, R36.2; no longer U6.27 (GPIO16)
- net KB_TX: now also J5.3 (Pin_3), R33.1, R37.2; no longer U6.28 (GPIO17)
- net LED_CAPS: now also RN1.1 (R1.1); no longer RN2.4 (R4.1)
- net LED_CHG: now also RN1.4 (R4.1); no longer RN1.3 (R3.1)
- net LED_DISK: now also RN1.2 (R2.1); no longer RN1.1 (R1.1)
- net LED_NUM: now also RN2.3 (R3.1); no longer RN2.2 (R2.1)
- net LED_PWM: now also R40.2
- net LED_PWR: now also RN1.3 (R3.1); no longer RN1.2 (R2.1)
- net LED_SCRL: now also RN2.4 (R4.1); no longer RN2.3 (R3.1)
- net LED_STBY: now also RN2.1 (R1.1); no longer RN1.4 (R4.1)
- net LED_WIFI: now also RN2.2 (R2.1); no longer RN2.1 (R1.1)
- net SCL: now also R39.2
- net SDA: now also R38.2
- net EC_BOOT: now reaches R17.1
- net at RN2.5 (R4.2): now also U12.7 (QH); no longer U6.14 (GPIO11)
- net at RN2.6 (R3.2): now also U12.6 (QG); no longer U6.13 (GPIO10)
- net at RN2.7 (R2.2): now also U12.5 (QF); no longer U6.12 (GPIO9)
- net at RN2.8 (R1.2): now also U12.4 (QE); no longer U6.11 (GPIO8)
- net at U6.6 (GPIO4): now also R32.2; no longer RN1.8 (R1.2)
- net at U6.7 (GPIO5): now also R33.2; no longer RN1.7 (R2.2)
- net at RN1.6 (R3.2): now also U12.3 (QD); no longer U6.8 (GPIO6)
- net at RN1.5 (R4.2): now also U12.15 (QA); no longer U6.9 (GPIO7)
- new net: Q1.1 (G), R40.1
- new net: J2.33 (LED_RTN), Q1.3 (D)
- new net: Q2.3 (D), R11.1
- new net: Q2.1 (G), R41.1
- new net: RN1.8 (R1.2), U12.1 (QB)
- new net: RN1.7 (R2.2), U12.2 (QC)
- new net EN_5V: U13.3 (QD)
- new net EN_ZERO: U13.1 (QB)
- new net SH2_OE: R42.1, U13.13 (~{OE})
- new net SH2_RST: R43.2, U13.10 (~{SRCLR})
- new net SH_CLK: U12.11 (SRCLK), U13.11 (SRCLK), U6.8 (GPIO6)
- new net SH_DIN: U12.14 (SER), U6.9 (GPIO7)
- new net SH_DOUT1: U12.9 (QH'), U13.14 (SER)
- new net SH_LATCH: U12.12 (RCLK), U13.12 (RCLK), U6.11 (GPIO8)
- new net SH_OE: R34.1, U12.13 (~{OE})
- new net SH_RST: R35.2, U12.10 (~{SRCLR})
- no-connect marks 11 -> 8
Other:
- note added: "TODO [x] i2c pullups [x] main [x] ec-kb [x] i2c/uart pin mix for ec-kb [x] led pwm [x] flip kb usb port [x] npn the kb boot away [x] shift reg for pm [x] shift reg for leds [x] second qwiic add 5v usb sensing to one rp2040 gpio pull one rpi gpio to the kb somewhere do a battery conn fp still pull one rpi gpio to batt conn pull one rp2040 gpio to batt conn omg one adc is version divider ec flash m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"
- note removed: "TODO i2c pullups main ec-kb i2c/uart pin mix for ec-kb led pwm omg one adc is version divider ec flash mode boot button mux switching power management vin/vbat switchover 5v step-up pi zero vin gating int usbc? pi zero usb pads hdmi port 5v pad second qwiic? power planes caps on adc one more adc? more caps on 3.3v? aux board header 3v3p usb shift reg for pm? could be cool shift reg for leds? cont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"
- moved on the sheet: C10, C11, C12, C13, C14, C46, C47, C9, J4, L1, L2, R1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

Commit message: sony_vaio_p_re: more work; power management PoC done
Parts:
- added C50, C51, C52, C53: 4u7, Capacitor_SMD:C_0805_2012Metric, symbol Device:C_Small
- added D2: SS34, Diode_SMD:D_SMA, symbol Device:D_Schottky_Small
- added ISET2, ISET3: x, Resistor_SMD:R_0402_1005Metric, symbol Device:R_Small
- added L4: 4u7, lib:L_Murata_23S4R7C, symbol Device:L_Small
- added PD2, PD3, PD4: 10K, Resistor_SMD:R_0402_1005Metric, symbol Device:R_Small
- added Q3: Q_PMOS_GSD, Package_TO_SOT_SMD:SOT-23, symbol Device:Q_PMOS_GSD
- added R44: 5V_FBU, Resistor_SMD:R_0402_1005Metric, symbol Device:R_Small
- added R45: 5V_FBD, Resistor_SMD:R_0402_1005Metric, symbol Device:R_Small
- added U10: MIC2876, Package_DFN_QFN:DFN-8-1EP_2x2mm_P0.5mm_EP0.6x1.2mm, symbol Regulator_Switching:MIC2290
- added U14, U15: SY6280, Package_TO_SOT_SMD:SOT-23-5, symbol sy6280_breakout-rescue:SY6280-sy6280
Connections:
- net +3.3V is gone; now on net +3V3: C15.1, C16.1, U3.11 (VDD5), U3.13 (VDD33)
- net +5VD: now also C52.1, C53.1, R44.2, U10.8 (OUT), U15.5 (IN)
- net EN_2V5: now also U13.15 (QA); no longer U13.2 (QC)
- net EN_3V3: now also U13.1 (QB); no longer U13.4 (QE)
- net EN_5V: now also U13.2 (QC), U10.6 (EN); no longer U13.3 (QD)
- net EN_ZERO: now also U13.7 (QH), PD2.1, U14.4 (EN); no longer U13.1 (QB)
- net GND: now also C50.2, C51.2, C52.2, C53.2, ISET2.2, ISET3.2, PD2.2, PD3.2, PD4.2, R45.1, U10.2 (PGND), U10.4 (AGND), U10.7 (PG), U10.9 (EP_GND), U14.2 (GND), U15.2 (GND)
- net VIN: now also C50.1, C51.1, D2.1 (K), L4.1, Q3.3 (D), U10.3 (VIN), U14.5 (IN)
- net EN_5VI: now reaches U13.6 (QG)
- net EN_5VI: now also PD3.1, U15.4 (EN)
- net +5V renamed VIN_PI
- net VIN_PI: now also U14.1 (OUT)
- new net: ISET3.1, U15.3 (ISET)
- new net: ISET2.1, U14.3 (ISET)
- new net +BATT: Q3.2 (S)
- new net 5V_FB: R44.1, R45.2, U10.5 (NC)
- new net 5V_INT: U15.1 (OUT)
- new net 5V_SW: L4.2, U10.1 (SW)
- new net 5V_VIN: D2.2 (A), PD4.1, Q3.1 (G)
Other:
- note added: "TODO [x] i2c pullups [x] main [x] ec-kb [x] i2c/uart pin mix for ec-kb [x] led pwm [x] flip kb usb port [x] npn the kb boot away [x] shift reg for pm [x] shift reg for leds [x] second qwiic power management [x] vin/vbat switchover [x] 5v step-up [x] pi zero vin gating [x] int usbc 5v regulator from VDC add internal usbc port add 5v usb sensing to one rp2040 gpio pull one rpi gpio to the kb somewh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"
- note removed: "TODO [x] i2c pullups [x] main [x] ec-kb [x] i2c/uart pin mix for ec-kb [x] led pwm [x] flip kb usb port [x] npn the kb boot away [x] shift reg for pm [x] shift reg for leds [x] second qwiic add 5v usb sensing to one rp2040 gpio pull one rpi gpio to the kb somewhere do a battery conn fp still pull one rpi gpio to batt conn pull one rp2040 gpio to batt conn omg one adc is version divider ec flash m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"

Commit message: sony_vaio_p_re: Some More Dev
Parts:
- added C54, C55, C56, C57: 4u7, Capacitor_SMD:C_0805_2012Metric, symbol Device:C_Small
- added C58: 100p, Capacitor_SMD:C_0402_1005Metric, symbol Device:C_Small
- added L5: 4u7, lib:L_Murata_23S4R7C, symbol Device:L_Small
- added Q4: Q_PMOS_GSD, Package_TO_SOT_SMD:SOT-23, symbol Device:Q_PMOS_GSD
- added R46: DC_FBU, Resistor_SMD:R_0402_1005Metric, symbol Device:R_Small
- added R47: DC_FBD, Resistor_SMD:R_0402_1005Metric, symbol Device:R_Small
- added U16: RT8078A, Package_DFN_QFN:DFN-10-1EP_3x3mm_P0.5mm_EP1.58x2.35mm, symbol Regulator_Switching:MIC2290
Connections:
- net +5VA: now also U9.1 (OUT); no longer U9.5 (IN)
- net +5VD: now also U9.5 (IN); no longer U9.1 (OUT)
- net +BATT: now also Q4.2 (S)
- net +VDC: now also C54.1, C56.1, U16.10 (PVIN), U16.7 (SVIN), U16.8 (PVIN), U16.9 (PVIN)
- net 5V_VIN: now also C55.1, C57.1, C58.1, L5.2, Q4.1 (G), R46.2
- net GND: now also C54.2, C55.2, C56.2, C57.2, R47.1, U16.11 (EP_GND)
- net VIN: now also Q4.3 (D)
- net EN_DC: now reaches U13.3 (QD)
- net EN_DC: now also U16.5 (NC)
- net EN_DCINR: now reaches U13.5 (QF)
- new net DC_FB: C58.2, R46.1, R47.2, U16.6 (FB)
- new net SW_DC: L5.1, U16.1 (LX), U16.2 (LX), U16.3 (LX)
Other:
- note added: "TODO [x] i2c pullups [x] main [x] ec-kb [x] i2c/uart pin mix for ec-kb [x] led pwm [x] flip kb usb port [x] npn the kb boot away [x] shift reg for pm [x] shift reg for leds [x] second qwiic power management [x] vin/vbat switchover [x] 5v step-up [x] pi zero vin gating [x] int usbc [x] 5v regulator from VDC BATTERY CHARGER ideal diode IC go through EN pins and check VDC reg 5V step-up charger sy62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"
- note removed: "TODO [x] i2c pullups [x] main [x] ec-kb [x] i2c/uart pin mix for ec-kb [x] led pwm [x] flip kb usb port [x] npn the kb boot away [x] shift reg for pm [x] shift reg for leds [x] second qwiic power management [x] vin/vbat switchover [x] 5v step-up [x] pi zero vin gating [x] int usbc 5v regulator from VDC add internal usbc port add 5v usb sensing to one rp2040 gpio pull one rpi gpio to the kb somewh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"
- moved on the sheet: D2, ISET1, PD1, PD4, Q3, U9

Commit message: sony_vaio_p_re: some more additions
Parts:
- removed R42: 4.7K, Resistor_SMD:R_0402_1005Metric, symbol Device:R
- added BT1: Battery, lib:BAT-SMD_CR1220-2ZX, symbol Device:Battery
- added C59: 100nF, Capacitor_SMD:C_0402_1005Metric, symbol Device:C
- added D3: 5V1, Diode_SMD:D_0805_2012Metric, symbol Device:D_Zener_Small
- added J7: AXK740347G_VAIO-P, lib:AXK750147G_VAIO-P, symbol AXK750147G:AXK750147G_VAIO-P
- added J8: RTC_BATT, Connector_JST:JST_SH_SM02B-SRSS-TB_1x02-1MP_P1.00mm_Horizontal, symbol Connector_Generic_MountingPin:Conn_01x02_MountingPin
- added Q11: SI4909, Package_SO:SO-8_3.9x4.9mm_P1.27mm, symbol Device:Q_Dual_PMOS_S1G1S2G2D2D2D1D1
- added Q7: 2N7002, Package_TO_SOT_SMD:SOT-23, symbol Device:Q_PMOS_GSD
- added R48: 5.1K, Resistor_SMD:R_0402_1005Metric, symbol Device:R_Small
- added R49: 5K1, Resistor_SMD:R_0402_1005Metric, symbol Device:R_Small
- added R52, R59: 1K8, Resistor_SMD:R_0402_1005Metric, symbol Device:R_Small
- added TP1, TP2: TestPoint, TestPoint:TestPoint_Pad_2.0x2.0mm, symbol Connector:TestPoint
- added U17: PCF85363ATT, Package_SO:TSSOP-8_3x3mm_P0.65mm, symbol Timer_RTC:PCF85363ATT
- added U18, U19, U20, U21: ESD, Package_TO_SOT_SMD:SOT-23-6, symbol Power_Protection:USBLC6-2SC6
- added U22, U23, U24, U25, U26, U27, U28: TPD4E02B04DQA, Package_SON:USON-10_2.5x1.0mm_P0.5mm, symbol Power_Protection:TPD4E02B04DQA
- added Y4: Crystal, Crystal:Crystal_SMD_TXC_9HT11-2Pin_2.0x1.2mm, symbol Device:Crystal
- U16: footprint Package_DFN_QFN:DFN-10-1EP_3x3mm_P0.5mm_EP1.58x2.35mm -> Package_TO_SOT_SMD:TSOT-23-6
Connections:
- net SH2_OE is gone; now on net GND: U13.13 (~{OE})
- net +3V3: now also U17.8 (VDD), U18.5 (VBUS), U19.5 (VBUS), U21.5 (VBUS)
- net +3V3E: now also U20.5 (VBUS)
- net +BATT: now also J7.1 (+VBATT1), J7.10 (+VBATT1), J7.11 (+VBATT1), J7.12 (+VBATT1), J7.13 (+VBATT1), J7.14 (+VBATT1), J7.15 (+VBATT1), J7.16 (+VBATT1), J7.17 (+VBATT1), J7.2 (+VBATT1), J7.3 (+VBATT1), J7.4 (+VBATT1), J7.5 (+VBATT1), J7.6 (+VBATT1), J7.7 (+VBATT1), J7.8 (+VBATT1), J7.9 (+VBATT1), TP2.1
- net +VDC: now also U16.4 (VIN), D3.1 (K), Q11.7 (D), Q11.8 (G), R59.1; no longer U16.10 (PVIN), U16.7 (SVIN), U16.8 (PVIN), U16.9 (PVIN)
- net 5V_VIN: now also Q11.5 (D), Q11.6 (G)
- net COL0: now also U23.4 (IO3), U23.7 (NC)
- net COL1: now also U27.5 (IO4), U27.6 (NC)
- net COL10: now also U25.4 (IO3), U25.7 (NC)
- net COL11: now also U22.4 (IO3), U22.7 (NC)
- net COL12: now also U27.2 (IO2), U27.9 (NC)
- net COL13: now also U23.1 (IO1), U23.10 (NC)
- net COL14: now also U25.5 (IO4), U25.6 (NC)
- net COL15: now also U27.1 (IO1), U27.10 (NC)
- net COL2: now also U26.5 (IO4), U26.6 (NC)
- net COL3: now also U22.1 (IO1), U22.10 (NC)
- net COL4: now also U25.1 (IO1), U25.10 (NC)
- net COL5: now also U25.2 (IO2), U25.9 (NC)
- net COL6: now also U22.2 (IO2), U22.9 (NC)
- net COL7: now also U27.4 (IO3), U27.7 (NC)
- net COL8: now also U23.2 (IO2), U23.9 (NC)
- net COL9: now also U22.5 (IO4), U22.6 (NC)
- net DC_FB: now also U16.1 (FB), R48.1; no longer C58.2, R46.1, R47.2, U16.6 (FB)
- net EN_2V5: now also U13.3 (QD); no longer U13.15 (QA)
- net EN_DC: now also U13.15 (QA), U16.2 (EN); no longer U13.3 (QD), U16.5 (NC)
- net EUSB1_N: now also U21.1 (I/O1)
- net EUSB1_P: now also U21.3 (I/O2)
- net GND: now also U16.3 (GND), BT1.2 (-), J7.23 (BATT_RTN), J7.24 (BATT_RTN), J7.25 (BATT_RTN), J7.26 (BATT_RTN), J7.27 (BATT_RTN), J7.28 (BATT_RTN), J7.29 (BATT_RTN), J7.30 (BATT_RTN), J7.31 (BATT_RTN), J7.32 (BATT_RTN), J7.33 (BATT_RTN), J7.34 (BATT_RTN), J7.35 (BATT_RTN), J7.36 (BATT_RTN), J7.37 (BATT_RTN), J7.38 (BATT_RTN), J7.39 (BATT_RTN), J7.40 (BATT_RTN), J8.2 (Pin_2), J8.MP (MountPin), Q7.3 (D), R49.2, TP1.1, U17.4 (VSS), U18.2 (GND), U19.2 (GND), U20.2 (GND), U21.2 (GND), U22.3 (G), U22.8 (G), U23.3 (G), U23.8 (G), U24.3 (G), U24.8 (G), U25.3 (G), U25.8 (G), U26.3 (G), U26.8 (G), U27.3 (G), U27.8 (G), U28.3 (G), U28.8 (G); no longer U16.11 (EP_GND)
- net GP22: now also U6.14 (GPIO11)
- net GP27: now also J7.22 (SYS_PRS#)
- net ROW0: now also U24.2 (IO2), U24.9 (NC)
- net ROW1: now also U24.5 (IO4), U24.6 (NC)
- net ROW2: now also U26.2 (IO2), U26.9 (NC)
- net ROW3: now also U26.4 (IO3), U26.7 (NC)
- net ROW4: now also U24.4 (IO3), U24.7 (NC)
- net ROW5: now also U26.1 (IO1), U26.10 (NC)
- net ROW6: now also U23.5 (IO4), U23.6 (NC)
- net ROW7: now also U24.1 (IO1), U24.10 (NC)
- net SCL: now also J7.20 (SMB_0CLK), U17.6 (SCL), U18.1 (I/O1)
- net SDA: now also J7.19 (SMB_0DATA), U17.5 (SDA), U18.6 (I/O1)
- net SW_DC: now also U16.5 (NC), C59.2; no longer U16.1 (LX), U16.2 (LX), U16.3 (LX)
- net USBi_DN: now also U20.1 (I/O1)
- net USBi_DP: now also U20.3 (I/O2)
- net VDC_BYPASS: now reaches U13.4 (QE)
- net VDC_BYPASS: now also Q7.1 (G), R49.1
- net RTC_INT: now reaches U6.12 (GPIO9)
- net RTC_INT: now also U17.7 (~{INTA})
- net 2040_G24: now reaches U6.36 (GPIO24)
- net 2040_G24: now also J7.21 (BATT1_PRS#), U18.4 (I/O2)
- net 2040_G25: now reaches U6.37 (GPIO25)
- net 2040_G25: now also J7.18 (BATT_ID), U18.3 (I/O2)
- net EN_DCINR: no longer names the net of U13.5 (QF)
- new net: C59.1, U16.6 (BOOT)
- new net: U17.2 (OSCO), Y4.1
- new net: U17.1 (OSCI), Y4.2
- new net: C58.2, R46.1, R47.2, R48.2
- new net: Q7.2 (S), R52.2
- new net: Q11.1 (S), Q11.3 (S)
- new net +VDC_G: D3.2 (A), Q11.2 (G), Q11.4 (G), R52.1, R59.2
- new net RTC_BATT: BT1.1 (+), J8.1 (Pin_1), U17.3 (VBAT)
Other:
- note added: "ESD"
- note added: "TODO [x] i2c pullups [x] main [x] ec-kb [x] i2c/uart pin mix for ec-kb [x] led pwm [x] flip kb usb port [x] npn the kb boot away [x] shift reg for pm [x] shift reg for leds [x] second qwiic power management [x] vin/vbat switchover [x] 5v step-up [x] pi zero vin gating [x] int usbc [x] 5v regulator from VDC [x] copy prev 5v regulator out BATTERY CHARGER [x] 5v vin fet bypass ideal diode IC go thro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"
- note added: "VIN bypass FET (for VIN = 5V)"
- note added: "VIN to 5V VIN regulator"
- note removed: "TODO [x] i2c pullups [x] main [x] ec-kb [x] i2c/uart pin mix for ec-kb [x] led pwm [x] flip kb usb port [x] npn the kb boot away [x] shift reg for pm [x] shift reg for leds [x] second qwiic power management [x] vin/vbat switchover [x] 5v step-up [x] pi zero vin gating [x] int usbc [x] 5v regulator from VDC BATTERY CHARGER ideal diode IC go through EN pins and check VDC reg 5V step-up charger sy62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"
- moved on the sheet: C33, C34, C35, C36, C37, C38, C39, C40, C41, C42, C43, C44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

Commit message: sony_vaio_p_re: hacking continues
Parts:
- removed U20: ESD, Package_TO_SOT_SMD:SOT-23-6, symbol Power_Protection:USBLC6-2SC6
- added C60: 100nF, Capacitor_SMD:C_0402_1005Metric, symbol Device:C
- added C61: 4u7, Capacitor_SMD:C_0603_1608Metric, symbol Device:C_Small
- added C62: 4u7, Capacitor_SMD:C_0805_2012Metric, symbol Device:C_Small
- added R42, R50: 4.7K, Resistor_SMD:R_0402_1005Metric, symbol Device:R
- added R51, R54, R56: 470K, Resistor_SMD:R_0402_1005Metric, symbol Device:R
- added R53, R55, R57: 100K, Resistor_SMD:R_0402_1005Metric, symbol Device:R
- added TP3: TestPoint, TestPoint:TestPoint_Pad_1.0x1.0mm, symbol Connector:TestPoint
- added U20: 24LC00, Package_SO:SOIC-8_3.9x4.9mm_P1.27mm, symbol Memory_EEPROM:24LC00
- added U29, U30: 74LVC1G17, Package_TO_SOT_SMD:SOT-23-5, symbol 74xGxx:74LVC1G17
- added U31: TPD4E02B04DQA, Package_SON:USON-10_2.5x1.0mm_P0.5mm, symbol Power_Protection:TPD4E02B04DQA
- U16: value RT8078A -> RT6255
Connections:
- net +3V3: now also R50.2, U20.1 (A0), U20.2 (A1), U20.3 (A2), U20.8 (VCC)
- net +3V3E: now also C61.2, C62.2, R42.2, R51.2, R54.2, R56.2, R57.2, U29.5 (VCC), U30.5 (VCC)
- net +5VA: now also R30.2
- net +5VD: no longer R30.2
- net 2040_G25: now also J7.21 (BATT1_PRS#), U18.4 (I/O2); no longer J7.18 (BATT_ID), U18.3 (I/O2)
- net 5V_EXT_EN: now also U6.35 (GPIO23); no longer U6.34 (GPIO22)
- net ADC2: now also R26.1, R27.2; no longer R28.1, R29.2
- net ADC3: no longer R30.1, R31.2
- net ADC4: now also R28.1, R29.2; no longer R26.1, R27.2
- net EC_BOOT: now also U30.4
- net GND: now also U20.4 (GND), U20.7 (WP), U29.3 (GND), U30.3 (GND), U31.3 (G), U31.8 (G)
- net GP25: no longer U6.16 (GPIO13)
- net GP26: now also U6.16 (GPIO13)
- net LCD_INS: now also U6.36 (GPIO24); no longer U6.35 (GPIO23)
- net L_FAULT: now also U6.27 (GPIO16); no longer U6.31 (GPIO20)
- net L_PWM: now also U6.28 (GPIO17); no longer U6.32 (GPIO21)
- net QSPI_E_SS: now also R42.1
- net QSPI_SS: now also R50.1
- net SCL: now also U20.6 (SCL)
- net SDA: now also U20.5 (SDA)
- net SHTDN: now also U6.31 (GPIO20)
- net SW_PWR: now also R55.1
- net SW_WIFI: now also R53.1
- net USBi_DN: now also U31.1 (IO1), U31.10 (NC)
- net USBi_DP: now also U31.2 (IO2), U31.9 (NC)
- net eUSB_SEL: now also U6.34 (GPIO22), R57.1
- net at R33.2: now also U6.6 (GPIO4); no longer U6.7 (GPIO5)
- net at R32.2: now also U6.7 (GPIO5); no longer U6.6 (GPIO4)
- net G10: now reaches U6.13 (GPIO10)
- net G10: now also TP3.1
- net EC_RUN: now reaches U6.26 (RUN)
- net EC_RUN: now also C60.2, R51.1
- removed net 2040_G24: J7.21 (BATT1_PRS#), U18.4 (I/O2), U6.36 (GPIO24)
- net ADC1 renamed 2040_G26
- net 2040_G26: now also J7.18 (BATT_ID), U18.3 (I/O2)
- net RUN renamed KB_RUN
- new net: C62.1, R55.2, R56.1, U29.2
- new net: C61.1, R53.2, R54.1, U30.2
- new net: C60.1, U29.4
- new net 5VA_DET: R30.1, R31.2, U6.32 (GPIO21)
Other:
- note added: "TODO [x] i2c pullups [x] main [x] ec-kb [x] i2c/uart pin mix for ec-kb [x] led pwm [x] flip kb usb port [x] npn the kb boot away [x] shift reg for pm [x] shift reg for leds [x] second qwiic [x] do a battery conn fp still [x] pull one rpi gpio to batt conn [x] pull one rp2040 gpio to batt conn [x] add battery testpoints [x] add qspi cs pullups [x] ec flash mode [x] rst on long pwr button press [x]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"
- note removed: "TODO [x] i2c pullups [x] main [x] ec-kb [x] i2c/uart pin mix for ec-kb [x] led pwm [x] flip kb usb port [x] npn the kb boot away [x] shift reg for pm [x] shift reg for leds [x] second qwiic power management [x] vin/vbat switchover [x] 5v step-up [x] pi zero vin gating [x] int usbc [x] 5v regulator from VDC [x] copy prev 5v regulator out BATTERY CHARGER [x] 5v vin fet bypass ideal diode IC go thro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"
- moved on the sheet: C33, R17, R32, R33, R36, R37, R38, R39, U1, U19, U28, U7
