File: Reverse-engineering/sony_vaio_p_re/vaio_re.kicad_sch (KiCad schematic)
At the start: 195 parts, among them IC1 SN75LVDS83B, J1 RPi_GPIO, J2 AXK750147G_VAIO-P, J3 AXK760347G_VAIO-P, J4 qwiic, J5 qwiic?, J6 20374-R30E-31, J7 AXK740347G_VAIO-P, J8 RTC_BATT, Q1 2N7002, Q11 SI4909, Q2 2N7002, Q3 Q_PMOS_GSD, Q4 Q_PMOS_GSD, Q7 2N7002, U1 AP2112K-3.3, U10 MIC2876, U12 74HC595, U13 74HC595, U14 SY6280, U15 SY6280, U16 RT6255, U17 PCF85363ATT, U18 ESD, U19 ESD, U2 PAM2306AYPAA, U20 24LC00, U21 ESD, U22 TPD4E02B04DQA, U23 TPD4E02B04DQA, U24 TPD4E02B04DQA, U25 TPD4E02B04DQA, U26 TPD4E02B04DQA, U27 TPD4E02B04DQA, U28 TPD4E02B04DQA, U29 74LVC1G17, U3 SL2.1A, U30 74LVC1G17, U31 TPD4E02B04DQA, U4 RP2040, U5 W25Q128JVS, U6 RP2040, U7 W25Q128JVS, U8 FSUSB42MUX, U9 SY6280, Y1 12MHz, Y2 ABM8-272-T3, Y3 ABM8-272-T3, Y4 Crystal

Commit message: sony_vaio_p_re: Some More Hacks
Parts:
- removed U18, U19: ESD, Package_TO_SOT_SMD:SOT-23-6, symbol Power_Protection:USBLC6-2SC6
- removed U28: TPD4E02B04DQA, Package_SON:USON-10_2.5x1.0mm_P0.5mm, symbol Power_Protection:TPD4E02B04DQA
- added C63, C75, C78: 1uF, Capacitor_SMD:C_0402_1005Metric, symbol Device:C
- added C64, C65, C66, C67, C69, C70, C71, C72, C73, C74, C76: 100nF, Capacitor_SMD:C_0402_1005Metric, symbol Device:C
- added C68, C77: 22uF, Capacitor_SMD:C_0805_2012Metric, symbol Device:C
- added ISET4: x, Resistor_SMD:R_0402_1005Metric, symbol Device:R_Small
- added J10, J9: EXP, Connector_FFC-FPC:Hirose_FH12-24S-0.5SH_1x24-1MP_P0.50mm_Horizontal, symbol Connector_Generic_MountingPin:Conn_01x24_MountingPin
- added JP1: A0, Jumper:SolderJumper-3_P1.3mm_Bridged12_Pad1.0x1.5mm, symbol Jumper:Jumper_3_Bridged12
- added JP2: A1, Jumper:SolderJumper-3_P1.3mm_Bridged12_Pad1.0x1.5mm, symbol Jumper:Jumper_3_Bridged12
- added JP3: A2, Jumper:SolderJumper-3_P1.3mm_Bridged12_Pad1.0x1.5mm, symbol Jumper:Jumper_3_Bridged12
- added PD5: 10K, Resistor_SMD:R_0402_1005Metric, symbol Device:R_Small
- added R58: 100K, Resistor_SMD:R_0402_1005Metric, symbol Device:R
- added R60, R61: 27, Resistor_SMD:R_0402_1005Metric, symbol Device:R
- added R62, R63: R, Resistor_SMD:R_0402_1005Metric, symbol Device:R
- added TP4: D+, TestPoint:TestPoint_Pad_1.0x1.0mm, symbol Connector:TestPoint
- added TP5: D-, TestPoint:TestPoint_Pad_1.0x1.0mm, symbol Connector:TestPoint
- added TP6: HDMI_POWER, TestPoint:TestPoint_Pad_1.0x1.0mm, symbol Connector:TestPoint
- added U32: PCF8574ATS, Package_SO:SSOP-20_4.4x6.5mm_P0.65mm, symbol Interface_Expansion:PCF8574ATS
- added U33, U34, U37: TPD4E02B04DQA, Package_SON:USON-10_2.5x1.0mm_P0.5mm, symbol esd_small:TPD4E02B04DQA
- added U35: ESD, Package_TO_SOT_SMD:SOT-23-6, symbol Power_Protection:USBLC6-2SC6
- added U36: SY6280, Package_TO_SOT_SMD:SOT-23-5, symbol sy6280_breakout-rescue:SY6280-sy6280
- R52: footprint Resistor_SMD:R_0402_1005Metric -> Resistor_SMD:R_0805_2012Metric
- U22, U23, U24, U25, U26, U27, U31: symbol Power_Protection:TPD4E02B04DQA -> esd_small:TPD4E02B04DQA
Connections:
- net +3.3VP: now also J9.17 (Pin_17), J9.18 (Pin_18)
- net +3V3: now also C67.1, C68.1, C69.1, C70.1, C71.1, C72.1, C73.1, C74.1, C75.1, C77.1, C78.1, J10.9 (Pin_9), J9.16 (Pin_16), JP1.1 (A), JP2.1 (A), JP3.1 (A), U32.5 (VDD), U35.5 (VBUS)
- net +3V3E: now also C66.1, C76.1, R58.2, R62.2
- net +5VD: now also U36.5 (IN)
- net +VDC: now also J10.19 (Pin_19), J10.20 (Pin_20), J10.21 (Pin_21), J10.22 (Pin_22), J10.23 (Pin_23), J10.24 (Pin_24)
- net 2040_G25: now also U37.1 (IO1), U37.10 (NC)
- net 2040_G26: now also U37.4 (IO3), U37.7 (NC)
- net 5VA_DET: now also U6.31 (GPIO20); no longer U6.32 (GPIO21)
- net 5V_EXT_EN: now also U6.32 (GPIO21); no longer U6.35 (GPIO23)
- net 5V_INT: now also J9.21 (Pin_21), J9.22 (Pin_22), J9.23 (Pin_23), J9.24 (Pin_24)
- net ADC2: now also C64.1
- net ADC3: now also R62.1, R63.2
- net ADC4: now also C65.1
- net EUSB0_N: now also U21.4 (I/O2), J9.10 (Pin_10)
- net EUSB0_P: now also U21.6 (I/O1), J9.9 (Pin_9)
- net EUSB1_N: now also U21.3 (I/O2), J9.12 (Pin_12); no longer U21.1 (I/O1)
- net EUSB1_P: now also U21.1 (I/O1), J9.11 (Pin_11); no longer U21.3 (I/O2)
- net GND: now also C63.2, C64.2, C65.2, C66.2, C67.2, C68.2, C69.2, C70.2, C71.2, C72.2, C73.2, C74.2, C75.2, C76.2, C77.2, C78.2, ISET4.2, J10.1 (Pin_1), J10.2 (Pin_2), J10.3 (Pin_3), J10.4 (Pin_4), J10.5 (Pin_5), J10.6 (Pin_6), J10.7 (Pin_7), J10.8 (Pin_8), J10.MP (MountPin), J9.1 (Pin_1), J9.19 (Pin_19), J9.2 (Pin_2), J9.20 (Pin_20), J9.3 (Pin_3), J9.4 (Pin_4), J9.MP (MountPin), JP1.3 (B), JP2.3 (B), JP3.3 (B), PD5.2, R63.1, U32.15 (VSS), U33.3 (G), U33.8 (G), U34.3 (G), U34.8 (G), U35.2 (GND), U36.2 (GND), U37.3 (G), U37.8 (G); no longer U8.10 (~{OE})
- net GP25: now also J9.15 (Pin_15), U32.1 (~{INT}), U35.4 (I/O2)
- net GP27: now also J10.13 (Pin_13), U34.5 (IO4), U34.6 (NC); no longer J7.22 (SYS_PRS#)
- net KB_RX: now also R61.2; no longer R15.1, U4.16 (GPIO13)
- net KB_TX: now also R60.1; no longer R16.1, U4.15 (GPIO12)
- net SCL: now also J10.18 (Pin_18), J9.14 (Pin_14), U32.2 (SCL), U35.6 (I/O1), U37.5 (IO4), U37.6 (NC)
- net SDA: now also J10.17 (Pin_17), J9.13 (Pin_13), U32.4 (SDA), U35.1 (I/O1), U37.2 (IO2), U37.9 (NC)
- net SHTDN: now also U6.30 (GPIO19); no longer U6.31 (GPIO20)
- net SH_CLK: now also J10.11 (Pin_11)
- net SH_LATCH: now also J10.12 (Pin_12)
- net USBIN_N: now also TP5.1
- net USBIN_P: now also TP4.1
- net VIN: now also C63.1
- net eUSB_SEL: now also U6.35 (GPIO23); no longer U6.34 (GPIO22)
- net LED_RTN: now reaches J2.33 (LED_RTN), Q1.3 (D)
- net SH_DOUT2: now reaches U13.9 (QH')
- net SH_DOUT2: now also J10.10 (Pin_10)
- net at U31.4 (IO3): now also U31.7 (NC)
- net at U31.5 (IO4): now also U31.6 (NC)
- new net: TP6.1, U36.1 (OUT)
- new net: ISET4.1, U36.3 (ISET)
- new net: PD5.1, U36.4 (EN)
- new net: R16.1, R60.2, U4.15 (GPIO12)
- new net: R15.1, R61.1, U4.16 (GPIO13)
- new net GPE_P0: J10.16 (Pin_16), U32.10 (P0), U34.1 (IO1), U34.10 (NC)
- new net GPE_P1: J10.15 (Pin_15), U32.11 (P1), U34.2 (IO2), U34.9 (NC)
- new net GPE_P2: J10.14 (Pin_14), U32.12 (P2), U34.4 (IO3), U34.7 (NC)
- new net GPE_P3: J7.22 (SYS_PRS#), U32.14 (P3), U35.3 (I/O2)
- new net GPE_P4: J9.5 (Pin_5), U32.16 (P4), U33.5 (IO4), U33.6 (NC)
- new net GPE_P5: J9.6 (Pin_6), U32.17 (P5), U33.4 (IO3), U33.7 (NC)
- new net GPE_P6: J9.7 (Pin_7), U32.19 (P6), U33.2 (IO2), U33.9 (NC)
- new net GPE_P7: J9.8 (Pin_8), U32.20 (P7), U33.1 (IO1), U33.10 (NC)
- new net IO_A0: JP1.2 (C), U32.6 (A0)
- new net IO_A1: JP2.2 (C), U32.7 (A1)
- new net IO_A2: JP3.2 (C), U32.9 (A2)
- new net eUSB_OE: R58.1, U6.34 (GPIO22), U8.10 (~{OE})
Other:
- note added: "2.5V (LCD) and 3.3V (external) regulator with 100% duty"
- note added: "5V header power swch"
- note added: "5V step-up with 100% duty"
- note added: "HDMI anti-OC"
- note added: "LCD backlight driver (6s4p)"
- note added: "Left USB power switch"
- note added: "Pi Zero power swch"
- note added: "Shift register (power EN pins)"
- moved on the sheet: C1, C10, C11, C12, C13, C14, C15, C16, C17, C18, C19, C2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

Commit message: sony_vaio_p_re: you might think it's insane how much I can fit on this board, but I feel like the insanity is only beginning
Parts:
- removed L4: 4u7, lib:L_Murata_23S4R7C, symbol Device:L_Small
- added C79, C80, C82, C83, C84, C85, C86: 1uF, Capacitor_SMD:C_0402_1005Metric, symbol Device:C
- added C87: 22uF, Capacitor_SMD:C_0805_2012Metric, symbol Device:C
- added L6: 1u, lib:L_Murata_23S4R7C, symbol Device:L_Small
- added R64: 0R, Resistor_SMD:R_0805_2012Metric, symbol Device:R_Small
- added U18, U19: LM66200, Package_SON:Texas_R-PUSON-N8_USON-8-1EP_1.6x2.1mm_P0.5mm_EP0.4x1.7mm, symbol Analog_Switch:MAX40200AUK
- C15, C16, C17: footprint Capacitor_SMD:C_0603_1608Metric -> Capacitor_SMD:C_0402_1005Metric
- H1, H2, H3, H4: symbol Mechanical:MountingHole -> Mechanical:MountingHole_Pad; now left out of the parts list
- R44: value 5V_FBU -> 5V_FB1
- R45: value 5V_FBD -> 5V_FB2
Connections:
- net +5VA: now also C85.1
- net +5VD: now also C79.1, C83.1, C86.1
- net +BATT: now also U18.6 (VIN2), U19.6 (VIN2)
- net 5V_INT: now also C84.1
- net 5V_SW: now also L6.2
- net 5V_VIN: now also U18.3 (VIN1), U19.3 (VIN1)
- net GND: now also H1.1, H2.1, H3.1, H4.1, C79.2, C80.2, C82.2, C83.2, C84.2, C85.2, C86.2, C87.2, U18.1 (GND), U18.4 (ON#), U18.5 (GND), U19.1 (GND), U19.4 (ON#), U19.5 (GND)
- net KB_RUN: now also U6.13 (GPIO10)
- net VIN: now also C82.1, R64.2, U19.2 (OUT), U19.7 (OUT); no longer C50.1, C51.1, U10.3 (VIN)
- net VIN_PI: now also C87.1
- net HDMI_POWER: now reaches TP6.1, U36.1 (OUT)
- net HDMI_POWER: now also C80.1
- net G18: now reaches U6.29 (GPIO18)
- net G18: now also TP3.1
- removed net G10: TP3.1, U6.13 (GPIO10)
- new net VIN_5VREG: C50.1, C51.1, L6.1, R64.1, U10.3 (VIN), U18.2 (OUT), U18.7 (OUT)
Other:
- note added: "Power path (5V boost IN)"
- note added: "Power path 1 (Zero => 3.3V, EC 3.3V, 3.3VP, 2.5V)"
- note added: "Power path 1 backup plan"
- moved on the sheet: C13, C14, C50, C51, C52, C53, J10, R44, R45, U10

Commit message: sony_vaio_p_re: moar good additions :3
Parts:
- added C81: 47nF, Capacitor_SMD:C_0402_1005Metric, symbol Device:C
- added C88, C89: 4u7, Capacitor_SMD:C_0603_1608Metric, symbol Device:C_Small
- added C90: 4u7, Capacitor_SMD:C_0805_2012Metric, symbol Device:C_Small
- added C91: 100nF, Capacitor_SMD:C_0402_1005Metric, symbol Device:C
- added D4: LED_Small, LED_SMD:LED_0603_1608Metric, symbol Device:LED_Small
- added L4: 1u, lib:L_Murata_23S4R7C, symbol Device:L_Small
- added PD10: 10K, Resistor_SMD:R_0402_1005Metric, symbol Device:R_Small
- added PD6: RISET, Resistor_SMD:R_0402_1005Metric, symbol Device:R_Small
- added PD7, PD8, PD9: RVSET, Resistor_SMD:R_0402_1005Metric, symbol Device:R_Small
- added U28: BQ2501x, Package_DFN_QFN:QFN-16-1EP_3x3mm_P0.5mm_EP1.7x1.7mm, symbol Battery_Management:BQ2501x
- added U38: MCP23S17_ML, Package_DFN_QFN:QFN-28-1EP_6x6mm_P0.65mm_EP4.25x4.25mm, symbol Interface_Expansion:MCP23S17_ML
- added U39, U40, U41, U42, U43: TPD4E02B04DQA, Package_SON:USON-10_2.5x1.0mm_P0.5mm, symbol esd_small:TPD4E02B04DQA
Connections:
- net +3V3E: now also C91.1
- net +BATT: now also C90.1, L4.2, U28.10 (BAT)
- net 5V_VIN: now also PD10.1, U28.1 (VBUS)
- net COL9: now also U39.5 (IO4), U39.6 (NC)
- net GND: now also C88.2, C89.2, C90.2, C91.2, PD6.2, PD7.2, PD8.2, U28.11 (GND), U28.12 (GND), U28.17 (GND), U39.3 (G), U39.8 (G), U40.3 (G), U40.8 (G), U41.3 (G), U41.8 (G), U42.3 (G), U42.8 (G), U43.3 (G), U43.4 (IO3), U43.7 (NC), U43.8 (G)
- net GPE_P3: now also D4.1 (K), U28.3 (STAT); no longer J7.22 (SYS_PRS#)
- net PS2_CLK: now also U42.2 (IO2), U42.9 (NC)
- net PS2_DAT: now also U42.1 (IO1), U42.10 (NC)
- net RX0+: now also U41.4 (IO3), U41.7 (NC)
- net RX0-: now also U41.5 (IO4), U41.6 (NC)
- net RX1+: now also U41.1 (IO1), U41.10 (NC)
- net RX1-: now also U41.2 (IO2), U41.9 (NC)
- net RX2+: now also U40.4 (IO3), U40.7 (NC)
- net RX2-: now also U40.5 (IO4), U40.6 (NC)
- net RXCLK+: now also U40.1 (IO1), U40.10 (NC)
- net RXCLK-: now also U40.2 (IO2), U40.9 (NC)
- net SW_LID: now also U43.1 (IO1), U43.10 (NC)
- net SW_PWR: now also U43.2 (IO2), U43.9 (NC)
- net SW_SP0: now also U39.1 (IO1), U39.10 (NC)
- net SW_SP1: now also U39.2 (IO2), U39.9 (NC)
- net SW_WIFI: now also U43.5 (IO4), U43.6 (NC)
- net VDC_BYPASS: now also U13.5 (QF); no longer U13.4 (QE)
- net LED_NUM_PRE: now reaches R16.1, R60.2, U4.15 (GPIO12)
- net LED_NUM_PRE: now also U39.4 (IO3), U39.7 (NC)
- net LED_CAPS_PRE: now reaches R15.1, R61.1, U4.16 (GPIO13)
- new net: PD7.1, U28.9 (VSET)
- new net: PD6.1, U28.4 (ICHG)
- new net: C81.1, U28.15 (BTST)
- new net: D4.2 (A), PD10.2
- new net: C88.1, U28.16 (PMID)
- new net: U42.4 (IO3), U42.7 (NC)
- new net: U42.5 (IO4), U42.6 (NC)
- new net BAT_TS: J7.22 (SYS_PRS#), PD8.1, PD9.2, U28.7 (TS)
- new net CHG_REGN: C89.1, PD9.1, U28.2 (REGN)
- new net EN_CHG: U13.4 (QE), U28.6 (~{EN})
- new net SW_CHG: C81.2, L4.1, U28.13 (SW), U28.14 (SW)
Other:
- moved on the sheet: C30, R10, R9, U22, U26, U27, U5
