File: Raspberry Pi stuff/zpui_shld_wg12864b/zpui_shld_wg12864b.kicad_pcb (KiCad board)
At the start: 2 copper layers, 65 x 56 mm, 51 parts, among them J1 I2C, J12 QWIIC, J2 LCD, J3 QWIIC, J5 Raspberry_Pi_2_3, Q1 2N7002, Q2 2N7002, Q3 2N7002, SW1 B, SW2 A, SW3 Up, SW4 Down, SW5 Right, SW6 Left, U1 74HC595, U2 M24C02-FMN, U3 MCP23008-xSO, U5 AP1117-33

Commit message: zpui_shld_wg12864b: v0.0
Parts:
- removed U3: MCP23008-xSO, Package_SO:SOIC-18W_7.5x11.6mm_P1.27mm
- added H1: MountingHole_Pad, MountingHole:MountingHole_3mm_Pad, F.Cu at (163.9, 84.1)
- added R17: 1K8, Resistor_SMD:R_0603_1608Metric, F.Cu at (186.2, 80.1)
- added R18: 1K8, Resistor_SMD:R_0603_1608Metric, F.Cu at (137.6, 86.8)
- added R20: 5K1, Resistor_SMD:R_0603_1608Metric, F.Cu at (140.1, 90.1)
- added R21: 5K1, Resistor_SMD:R_0603_1608Metric, F.Cu at (184.6, 76.4)
- added R22: 5K1, Resistor_SMD:R_0603_1608Metric, B.Cu at (180.4, 97.1)
- added RV2: 10K, Potentiometer_SMD:Potentiometer_Bourns_3314J_Vertical, F.Cu at (134.2, 80.7)
- added U4: PCF8574, Package_SO:SOIC-16W_7.5x10.3mm_P1.27mm, B.Cu at (174.7, 86.3)
- moved TP4 12.6 mm to (158.3, 77.3)
- moved C1 12.5 mm to (170.0, 79.2), turned to 90 degrees
- moved JP1 10.1 mm to (183.9, 81.6)
- moved JP3 8.04 mm to (183.8, 86.4)
- moved JP2 7.67 mm to (183.9, 84.1)
- moved TP1 4.01 mm to (158.2, 89.7)
- moved TP2 4.01 mm to (158.2, 85.6)
- moved TP3 4.01 mm to (158.3, 81.3)
- moved R15 2.72 mm to (176.4, 77.1)
- renumbered TP0 to TP4
Connections:
- Q1 pad 1: LED_DRV -> Net-(Q1-G)
- Q2 pad 1: SH_CS -> Net-(Q2-G)
- R16 pad 1: SH_CS -> Net-(Q2-G)
Routing:
- net MCP_INT: track 11.0 -> 30.6 mm
- net RT_BTN: track 37.6 -> 53.0 mm
- net DN_BTN: track 40.0 -> 54.9 mm
- net A_BTN: track 46.5 -> 58.8 mm
- net Net-(U4-P7): track 5.20 -> 14.3 mm
- net SDA: track 82.3 -> 90.6 mm
- net SCL: track 75.5 -> 83.5 mm
- net Net-(U4-P6): track 5.03 -> 12.9 mm
- net Net-(Q2-G): track 0.00 -> 5.20 mm, vias 0 -> 1
- net Net-(Q1-G): track 0.00 -> 3.60 mm
- net UP_BTN: track 48.0 -> 51.5 mm
- net LT_BTN: track 53.0 -> 56.2 mm
- net SH_CS: track 58.2 -> 55.1 mm, vias 2 -> 1
- net GND: track 19.3 -> 16.2 mm, vias 49 -> 42
- net LED_DRV: track 48.1 -> 45.1 mm
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
Commit message: zpui_shld_wg12864b: v1
Parts:
- added G***: LOGO, LOGO, F.Cu at (162.3, 82.0)
- added G***: LOGO, LOGO, F.Cu at (139.0, 108.2)
- added G***: LOGO, LOGO, B.Cu at (158.3, 100.4)
- added G***: LOGO, LOGO, B.Cu at (139.0, 98.3)
- added J4: USB_C_Receptacle_USB2.0_16P, Connector_USB:USB_C_Receptacle_HRO_TYPE-C-31-M-12, F.Cu at (191.3, 87.2)
- added R23: 5K1, Resistor_SMD:R_0603_1608Metric, F.Cu at (185.1, 85.5)
- added R24: 5K1, Resistor_SMD:R_0603_1608Metric, F.Cu at (185.0, 88.4)
- added R25: 0/F, Resistor_SMD:R_0805_2012Metric, F.Cu at (187.3, 94.6)
- added U3: CH340C, Package_SO:SOIC-16_3.9x9.9mm_P1.27mm, B.Cu at (191.8, 108.5)
- R12: footprint Resistor_SMD:R_0603_1608Metric -> zpui_shld_wg12864b:R_0603_1608Metric_Jumper
- SW1: value B -> A
- SW2: value A -> B
- moved R17 1.68 mm to (184.7, 79.5)
- moved JP3 0.20 mm to (183.9, 86.6)
- moved C9 0.10 mm to (186.5, 99.8)
- moved R13 0.09 mm to (175.2, 99.6)
- turned R19 to 90 degrees
Connections:
- C5 pad 1: +5VL -> +5V
- J5 pad 29: A_BTN -> B_BTN
- J5 pad 32: B_BTN -> A_BTN
- R19 pad 1: +5VL -> +5V
- R19 pad 2: +5V -> +5VL
- SW1 pad 1: B_BTN -> A_BTN
- SW2 pad 1: A_BTN -> B_BTN
- U4 pad 4: B_BTN -> A_BTN
- U4 pad 5: A_BTN -> B_BTN
- U5 pad 3: +5VL -> +5V
Routing:
- net D-: track 0.00 -> 28.9 mm, vias 0 -> 1
- net D+: track 0.00 -> 28.3 mm, vias 0 -> 1
- net +3V3: track 194.9 -> 217.1 mm, vias 5 -> 7
- net TXD: track 0.00 -> 21.5 mm
- net +5VL: track 106.9 -> 86.2 mm, vias 1 -> 0
- net +5V: track 1.55 -> 21.9 mm, vias 0 -> 1
- net RXD: track 0.00 -> 19.8 mm
- net +5VP: track 0.00 -> 14.1 mm
- net A_BTN: track 58.8 -> 64.9 mm
- net B_BTN: track 64.8 -> 60.7 mm
- net SCL: track 83.5 -> 80.1 mm
- net LED_DRV: track 45.1 -> 46.8 mm
- net Net-(J4-CC2): track 0.00 -> 1.47 mm
- net Net-(J4-CC1): track 0.00 -> 1.45 mm
- net SDA: track 90.6 -> 89.3 mm
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- added copper zone on F.Cu, net +5V
- added copper zone on F.Cu, net +5VD
Other:
- board text added: "Bronze tribute"
- board text added: "CS invert bypass"
- board text added: "USB-UART"
- board text added: "contrast"
- board text added: "extra reg for {dblquote}3.3v off when off{dblquote} Pis"
- board text added: "funni display connector"
- board text added: "hackmods panel v1"
- board text added: "many I2C much wow"
- board text added: "oh hey look a civilian airliner"
- board text added: "trade CS2 for MPR_INT"
- board text added: "two extra IOs for 26-pin Pi"
- board text added: "{dblquote}26-pin header Pi{dblquote} contingencies"
- board text added: "{dblquote}free up SPI{dblquote} contingency"
