File: Raspberry Pi stuff/zpn_devboard/zpn_devboard.kicad_pcb (KiCad board)
At the start: 2 copper layers, 150 x 100 mm, 95 parts, among them J1 SH 4P, J2 SH 4P, J3 Raspberry_Pi_2_3, J4 USB, Q1 2N7002, U1 FSUSB42MUX, U10 SL2.1A, U11 SY6280, U12 MCP23S17_ML, U2 W25Q128JVS, U3 74LVC1G17, U4 74LVC1G17, U5 FSUSB42MUX, U6 RP2040, U7 AP2112K-3.3, U8 TPD4E02B04DQA, U9 74HC595, Y1 12MHz, Y2 12MHz

Commit message: zpn_devboard: v0; needs review before ordering
Parts:
- removed C11, C25, C26: 100nF, Capacitor_SMD:C_0402_1005Metric
- removed C5: 4.7uF, Capacitor_SMD:C_0805_2012Metric
- removed C8: 4.7uF, Capacitor_SMD:C_0603_1608Metric
- removed R29: NC, Resistor_SMD:R_0603_1608Metric
- removed the REF** at (199.0, 105.0)
- removed RN1, RN2: 1.8K, Resistor_SMD:R_Array_Concave_4x0402
- removed TP1: TestPoint, TestPoint:TestPoint_Pad_1.0x1.0mm
- removed TP2: D+, TestPoint:TestPoint_Pad_1.0x1.0mm
- removed TP3: D-, TestPoint:TestPoint_Pad_1.0x1.0mm
- removed U9: 74HC595, Package_SO:SO-16_3.9x9.9mm_P1.27mm
- added C35: 100p, Capacitor_SMD:C_0603_1608Metric, F.Cu at (110.0, 145.5)
- added C36: 100p, Capacitor_SMD:C_0603_1608Metric, F.Cu at (107.3, 136.0)
- added C37: 1uF, Capacitor_SMD:C_0402_1005Metric, F.Cu at (133.4, 60.7)
- added C38: 1uF, Capacitor_SMD:C_0402_1005Metric, F.Cu at (129.1, 63.1)
- added C39: 1uF, Capacitor_SMD:C_0402_1005Metric, F.Cu at (111.6, 51.1)
- added C40: 1uF, Capacitor_SMD:C_0402_1005Metric, F.Cu at (106.5, 62.6)
- added C41: 1uF, Capacitor_SMD:C_0402_1005Metric, F.Cu at (115.8, 63.0)
- added C42: 1uF, Capacitor_SMD:C_0402_1005Metric, F.Cu at (104.5, 116.7)
- added C43: 1uF, Capacitor_SMD:C_0402_1005Metric, F.Cu at (109.4, 116.8)
- added C44: 1uF, Capacitor_SMD:C_0402_1005Metric, F.Cu at (104.0, 130.5)
- added C45: 1uF, Capacitor_SMD:C_0402_1005Metric, F.Cu at (108.9, 133.9)
- added C46: 1uF, Capacitor_SMD:C_0402_1005Metric, F.Cu at (168.8, 76.3)
- added C47: 1uF, Capacitor_SMD:C_0402_1005Metric, F.Cu at (167.8, 80.0)
- added C48: 100nF, Capacitor_SMD:C_0402_1005Metric, F.Cu at (119.0, 73.6)
- added D2: LED 0603, LED_SMD:LED_0805_2012Metric_Pad1.15x1.40mm_HandSolder, F.Cu at (175.9, 55.0)
- added D3: LED 0603, LED_SMD:LED_0805_2012Metric_Pad1.15x1.40mm_HandSolder, F.Cu at (185.0, 66.6)
- added D4: SS34, Diode_SMD:D_SMA, F.Cu at (181.0, 53.4)
- added F1: 2A PTC, Fuse:Fuse_1206_3216Metric, F.Cu at (183.2, 61.0)
- added H1: mPCIe standoff, zpn_devboard:Standoff_M3_M2.5_Paste, F.Cu at (129.8, 80.7)
- added H2: mPCIe standoff, zpn_devboard:Standoff_M3_M2.5_Paste, F.Cu at (129.8, 104.9)
- added J10: b, Connector_PinHeader_2.54mm:PinHeader_1x08_P2.54mm_Vertical, F.Cu at (141.0, 76.2)
- added J11: r, Connector_PinHeader_2.54mm:PinHeader_1x10_P2.54mm_Vertical, F.Cu at (161.3, 53.3)
- added J12: Sn, Connector_PinHeader_2.54mm:PinHeader_1x04_P2.54mm_Vertical, F.Cu at (129.8, 136.5)
- added J13: KP, Connector_PinHeader_2.54mm:PinHeader_2x04_P2.54mm_Vertical, F.Cu at (128.4, 110.4)
- added J14: SH 4P, Connector_JST:JST_SH_SM04B-SRSS-TB_1x04-1MP_P1.00mm_Horizontal, F.Cu at (114.5, 146.7)
- added J15: SH 4P, Connector_JST:JST_SH_SM04B-SRSS-TB_1x04-1MP_P1.00mm_Horizontal, F.Cu at (122.2, 146.7)
- added J16: SH 4P, Connector_JST:JST_SH_BM04B-SRSS-TB_1x04-1MP_P1.00mm_Vertical, F.Cu at (162.1, 131.6)
- added J17: FPC 24P 0.5mm, Connector_FFC-FPC:Hirose_FH12-24S-0.5SH_1x24-1MP_P0.50mm_Horizontal, F.Cu at (105.8, 105.7)
- added J18: USB_C_Receptacle_USB2.0_16P, Connector_USB:USB_C_Receptacle_HRO_TYPE-C-31-M-12, F.Cu at (195.7, 76.0)
- added J19: SIM_Card, zpn_devboard:MICROSIM_6P_SMD_HOLDER, F.Cu at (109.6, 78.6)
- added J20: Conn_01x01, Connector_PinHeader_2.54mm:PinHeader_1x01_P2.54mm_Vertical, F.Cu at (199.0, 105.0)
- added J21: Conn_01x04, Connector_PinHeader_2.54mm:PinHeader_1x04_P2.54mm_Vertical, F.Cu at (152.9, 82.7)
- added J22: Battery, Connector_JST:JST_PH_S2B-PH-SM4-TB_1x02-1MP_P2.00mm_Horizontal, F.Cu at (193.2, 57.3)
- added J5: USB_C_Receptacle_USB2.0_16P, zpn_devboard:USB-TYPE-C-TH_TYPEC-300D-BCP16H100, F.Cu at (142.0, 109.6)
- added J6: USB_C_Host_a, Connector_USB:USB_C_Receptacle_HRO_TYPE-C-31-M-12, F.Cu at (103.8, 142.0)
- added J7: Bus_PCI_Express_Mini, Connector_PCBEdge:BUS_PCI_Express_Mini_Dual, F.Cu at (117.7, 56.8)
- added J8: USB_C_Receptacle_USB2.0_16P, Connector_USB:USB_C_Receptacle_HRO_TYPE-C-31-M-12, F.Cu at (103.8, 123.4)
- added J9: l, Connector_PinHeader_2.54mm:PinHeader_1x10_P2.54mm_Vertical, F.Cu at (138.4, 53.3)
- added N1: SK6805, zpn_devboard:SK6805-EC14, F.Cu at (159.4, 103.8)
- added N2: SK6805, zpn_devboard:SK6805-EC14, F.Cu at (101.0, 131.6)
- added Q2: BSS138, Package_TO_SOT_SMD:SOT-23, F.Cu at (173.9, 61.1)
- added Q3: BSS138, Package_TO_SOT_SMD:SOT-23, F.Cu at (173.9, 64.4)
- added R35: 5.1K, Resistor_SMD:R_0402_1005Metric, F.Cu at (136.3, 113.4)
- added R37: 27, Resistor_SMD:R_0402_1005Metric, F.Cu at (119.9, 76.2)
- added R38: 5.1K, Resistor_SMD:R_0402_1005Metric, F.Cu at (137.3, 113.3)
- added R39: 0R, Resistor_SMD:R_0402_1005Metric, F.Cu at (108.9, 134.9)
- added R40: 0R, Resistor_SMD:R_0603_1608Metric, F.Cu at (107.3, 134.1)
- added R41: 56K, Resistor_SMD:R_0402_1005Metric, F.Cu at (109.4, 126.0)
- added R42: 56K, Resistor_SMD:R_0402_1005Metric, F.Cu at (109.6, 121.5)
- added R43: 47R, Resistor_SMD:R_0402_1005Metric, F.Cu at (184.3, 135.9)
- added R44: 47R, Resistor_SMD:R_0402_1005Metric, F.Cu at (187.4, 138.3)
- added R45: 47R, Resistor_SMD:R_0402_1005Metric, F.Cu at (182.3, 134.1)
- added R46: 47R, Resistor_SMD:R_0402_1005Metric, F.Cu at (180.4, 132.5)
- added R47: 47R, Resistor_SMD:R_0402_1005Metric, F.Cu at (182.9, 138.7)
- added R48: 47R, Resistor_SMD:R_0402_1005Metric, F.Cu at (185.2, 141.2)
- added R49: 5.1K, Resistor_SMD:R_0402_1005Metric, F.Cu at (146.1, 120.3)
- added R50: 5.1K, Resistor_SMD:R_0402_1005Metric, F.Cu at (146.1, 119.4)
- added R51: 12k, Resistor_SMD:R_0402_1005Metric, F.Cu at (130.7, 65.6)
- added R52: 20K, Resistor_SMD:R_0402_1005Metric, F.Cu at (132.6, 65.7)
- added R53: 1.8K, Resistor_SMD:R_0402_1005Metric, F.Cu at (183.5, 64.4)
- added R55: 12k, Resistor_SMD:R_0402_1005Metric, F.Cu at (108.5, 114.2)
- added R56: 20K, Resistor_SMD:R_0402_1005Metric, F.Cu at (106.5, 114.2)
- added R57: 12k, Resistor_SMD:R_0402_1005Metric, F.Cu at (110.1, 129.8)
- added R58: 20K, Resistor_SMD:R_0402_1005Metric, F.Cu at (105.3, 130.0)
- added R59: 0R, zpn_devboard:R_0603_1608Metric_Jumper_Pwr, F.Cu at (119.8, 137.0)
- added R60: 0R, zpn_devboard:R_0603_1608Metric_Jumper_Pwr, F.Cu at (119.9, 138.6)
- added R61: NC, Resistor_SMD:R_0603_1608Metric, F.Cu at (122.8, 137.0)
- added R62: NC, Resistor_SMD:R_0603_1608Metric, F.Cu at (122.9, 138.6)
- added R63: 12K, Resistor_SMD:R_0402_1005Metric, F.Cu at (172.1, 79.9)
- added R64: 20K, Resistor_SMD:R_0402_1005Metric, F.Cu at (170.2, 76.7)
- added R65: 5.1K, Resistor_SMD:R_0402_1005Metric, F.Cu at (189.1, 78.0)
- added R67: 5.1K, Resistor_SMD:R_0402_1005Metric, F.Cu at (189.1, 73.4)
- added REF**: Hirose_FH12-24S-0.5SH_1x24-1MP_P0.50mm_Horizontal, Connector_FFC-FPC:Hirose_FH12-24S-0.5SH_1x24-1MP_P0.50mm_Horizontal, F.Cu at (90.6, 105.7)
- added SW1: bootton, zpn_devboard:SW-SMD_4P-L2.8-W1.9-P1.20-LS3.0, F.Cu at (140.5, 101.2)
- added SW2: resetton, zpn_devboard:SW-SMD_4P-L2.8-W1.9-P1.20-LS3.0, F.Cu at (156.0, 85.5)
- added TP4: TestPoint, zpn_devboard:TestPoint_Pad_1.0x1.0mm, F.Cu at (109.1, 143.2)
- added TP5: TestPoint, zpn_devboard:TestPoint_Pad_1.0x1.0mm, F.Cu at (109.1, 140.3)
- added TP6: TestPoint, zpn_devboard:TestPoint_Pad_1.0x1.0mm, F.Cu at (117.2, 67.3)
- added U13: FUSB302BMPX, Package_DFN_QFN:WQFN-14-1EP_2.5x2.5mm_P0.5mm_EP1.45x1.45mm, F.Cu at (104.8, 134.1)
- added U14: ESP32-C6-WROOM-1, PCM_Espressif:ESP32-C6-WROOM-1, F.Cu at (148.7, 139.7)
- added U15: SY6280, Package_TO_SOT_SMD:SOT-23-5, F.Cu at (131.8, 63.4)
- added U16: SY6280, Package_TO_SOT_SMD:SOT-23-5, F.Cu at (107.0, 116.3)
- added U17: SY6280, Package_TO_SOT_SMD:SOT-23-5, F.Cu at (108.1, 131.1)
- added U18: TPD4E02B04DQA, Package_SON:USON-10_2.5x1.0mm_P0.5mm, F.Cu at (126.0, 142.6)
- added U19: TPD4E02B04DQA, Package_SON:USON-10_2.5x1.0mm_P0.5mm, F.Cu at (120.3, 66.0)
- added U20: SY6280, Package_TO_SOT_SMD:SOT-23-5, F.Cu at (169.8, 79.2)
- C1: value 10uF -> 1uF; footprint Capacitor_SMD:C_0603_1608Metric -> Capacitor_SMD:C_0402_1005Metric
- D1: value D_Schottky_Small -> LED 0603; footprint Diode_SMD:D_SOD-323 -> LED_SMD:LED_0805_2012Metric_Pad1.15x1.40mm_HandSolder
- Q1: value 2N7002 -> BSS138
- R1: value 100K -> 5.1K
- R18: value 5.1K -> 47R
- R19: value 5.1K -> NP
- R2: value 470K -> 5.1K
- R20, R4, R9: value 470K -> 1.8K
- R21: value 100K -> 0R; footprint Resistor_SMD:R_0402_1005Metric -> zpn_devboard:R_0603_1608Metric_Jumper_Pwr
- R22, R23: value 20K -> 5.1K
- R24: value 20K -> NP; footprint Resistor_SMD:R_0402_1005Metric -> Resistor_SMD:R_0603_1608Metric
- R25: value 20K -> 0R; footprint Resistor_SMD:R_0402_1005Metric -> zpn_devboard:R_0603_1608Metric_Jumper_Pwr
- R26: value 470K -> 0R; footprint Resistor_SMD:R_0402_1005Metric -> zpn_devboard:R_0603_1608Metric_Jumper_Pwr
- R27: value 100K -> NP; footprint Resistor_SMD:R_0402_1005Metric -> Resistor_SMD:R_0603_1608Metric
- R3: value 100K -> 56K
- R36: value NC -> 27; footprint Resistor_SMD:R_0603_1608Metric -> Resistor_SMD:R_0402_1005Metric
- U3: value 74LVC1G17 -> CH340C; footprint Package_TO_SOT_SMD:SOT-23-5 -> Package_SO:SOIC-16_3.9x9.9mm_P1.27mm
- U4: value 74LVC1G17 -> TP4056; footprint Package_TO_SOT_SMD:SOT-23-5 -> Package_SO:SOIC-8-1EP_3.9x4.9mm_P1.27mm_EP2.29x3mm
- moved U8 131.4 mm to (124.4, 121.8)
- moved R36 96.4 mm to (121.0, 76.2), turned to -90 degrees
- moved C16 83.6 mm to (142.3, 82.7)
- moved C14 81.9 mm to (143.5, 83.1), turned to 90 degrees
- moved C23 79.9 mm to (148.0, 98.3), turned to 45 degrees
- moved C2 73.1 mm to (182.2, 57.4)
- moved D1 70.9 mm to (173.8, 55.0), turned to 90 degrees
- moved C1 70.2 mm to (180.8, 66.3), turned to 180 degrees
- moved R1 70.1 mm to (153.4, 85.1), turned to 90 degrees
- moved U4 65.8 mm to (179.4, 61.9), turned to 90 degrees
- moved R23 60.5 mm to (171.0, 62.6)
- moved R18 58.4 mm to (171.0, 60.3)
- moved U3 54.8 mm to (182.6, 76.1), turned to 90 degrees
- moved R22 54.3 mm to (176.3, 64.4), turned to -90 degrees
- moved R21 53.4 mm to (176.1, 66.5), turned to 180 degrees
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Connections:
- C1 pad 1: +VSW -> VBUS_chg
- C2 pad 1: GND -> +BATT
- C2 pad 2: +3V3 -> GND
- C29 pad 1: +3V3_2 -> +3V3
- C30 pad 1: +3V3_2 -> +3V3
- C33 pad 1: +3V3_2 -> +3V3_w
- D1 pad 1: +VSW -> Net-(D1-K)
- D1 pad 2: +3V3 -> VBUS_chg
- J3 pad 1: +3V3 -> +3V3_2
- J3 pad 19: unconnected-(J3-MOSI0/GPIO10-Pad19) -> S0I
- J3 pad 2: unconnected-(J3-5V-Pad2) -> VIN_Pi_o
- J3 pad 21: unconnected-(J3-MISO0/GPIO9-Pad21) -> S0O
- J3 pad 23: unconnected-(J3-SCLK0/GPIO11-Pad23) -> S0C
- J3 pad 24: unconnected-(J3-~{CE0}/GPIO8-Pad24) -> S0E0
- J3 pad 26: unconnected-(J3-~{CE1}/GPIO7-Pad26) -> S0E1
- J3 pad 29: unconnected-(J3-GCLK1/GPIO5-Pad29) -> INT
- J3 pad 4: unconnected-(J3-5V-Pad4) -> VIN_Pi_o
- J3 pad 7: Net-(J3-GCLK0/GPIO4) -> Pi_INT
- R1 pad 1: SW_PWR -> EC_RUN
- R1 pad 2: Net-(C5-Pad1) -> +3V3E
- R18 pad 1: SH_OE -> CHG_DIS
- R18 pad 2: GND -> Net-(Q2-G)
- R19 pad 1: +3V3E -> VBUS_chg
- R19 pad 2: SH_RST -> /TEMP
- R2 pad 1: Net-(C5-Pad1) -> GND
- R2 pad 2: +3V3E -> Net-(Q2-G)
- R20 pad 1: ADC2 -> /PROG
- R20 pad 2: +VDC -> GND
- R21 pad 1: GND -> /TEMP
- R21 pad 2: ADC2 -> GND
- R22 pad 1: ADC4 -> /PROG
- R22 pad 2: /VIN -> Net-(Q3-D)
- R23 pad 2: ADC4 -> CHG_PWR
- R24 pad 1: 5VA_DET -> Net-(J22-Pin_2)
- R24 pad 2: +5VA -> Net-(F1-Pad1)
- R25 pad 1: GND -> Net-(J22-Pin_2)
- R25 pad 2: 5VA_DET -> GND
- R26 pad 1: ADC3 -> Net-(J22-Pin_1)
- R26 pad 2: +3V3E -> Net-(F1-Pad1)
- R27 pad 1: GND -> Net-(J22-Pin_1)
- R27 pad 2: ADC3 -> GND
- R3 pad 1: SW_WIFI -> Net-(Q2-D)
- R3 pad 2: Net-(C8-Pad1) -> VBUS_chg
- R33 pad 1: 5V_EXT_EN -> ESP_PWR_EN
- R36 pad 1: Net-(J3-GCLK0/GPIO4) -> EC_HwSCL_m
- R36 pad 2: INT -> EC_HwSCL
- R4 pad 1: Net-(C8-Pad1) -> Net-(D1-K)
- R4 pad 2: +3V3E -> Net-(U4-~{CHRG})
- R9 pad 1: EC_RUN -> Net-(D2-K)
- R9 pad 2: +3V3E -> Net-(U4-~{STDBY})
- U10 pad 11: +3V3_2 -> +3V3
- U10 pad 13: +3V3_2 -> +3V3
- U10 pad 3: unconnected-(U10-DM3-Pad3) -> /USBc_DN
- U10 pad 4: unconnected-(U10-DP3-Pad4) -> /USBc_DP
- U10 pad 5: unconnected-(U10-DM2-Pad5) -> /USBb_DN
- U10 pad 6: unconnected-(U10-DP2-Pad6) -> /USBb_DP
- U10 pad 7: unconnected-(U10-DM1-Pad7) -> /USBa_DN
- U10 pad 8: unconnected-(U10-DP1-Pad8) -> /USBa_DP
- U11 pad 1: +3V3_2 -> +3V3_w
- U11 pad 4: 5V_EXT_EN -> ESP_PWR_EN
- U12 pad 1: unconnected-(U12-GPB4-Pad1) -> ESP_EN
- U12 pad 17: /GP_MDM1 -> /GP_KP1
- U12 pad 18: /GP_MDM2 -> /GP_KP2
- U12 pad 19: /GP_MDM3 -> /GP_KP3
- U12 pad 2: unconnected-(U12-GPB5-Pad2) -> ESP_PWR_EN
- U12 pad 20: unconnected-(U12-GPA3-Pad20) -> /GP_KP4
- U12 pad 21: unconnected-(U12-GPA4-Pad21) -> /GP_KP5
- U12 pad 22: unconnected-(U12-GPA5-Pad22) -> /GP_KP6
- U12 pad 23: unconnected-(U12-GPA6-Pad23) -> /GP_MDM1
- U12 pad 24: unconnected-(U12-GPA7-Pad24) -> /GP_MDM2
- U12 pad 25: unconnected-(U12-GPB0-Pad25) -> /GP_MDM3
- U12 pad 26: unconnected-(U12-GPB1-Pad26) -> /GP_USBC2
- U12 pad 27: unconnected-(U12-GPB2-Pad27) -> /GP_USBC1
- U12 pad 28: unconnected-(U12-GPB3-Pad28) -> VBUS_DBG_DET
- U3 pad 1: unconnected-(U3-NC-Pad1) -> GND
- U3 pad 2: Net-(C5-Pad1) -> RXD
- U3 pad 3: GND -> TXD
- U3 pad 4: Net-(C11-Pad1) -> +3V3_2
- U3 pad 5: +3V3E -> /USBf_DP
- U4 pad 1: unconnected-(U4-NC-Pad1) -> /TEMP
- U4 pad 2: Net-(C8-Pad1) -> /PROG
- U4 pad 4: /EC_BOOT -> VBUS_chg
- U4 pad 5: +3V3E -> +BATT
- U6 pad 11: unconnected-(U6-GPIO8-Pad11) -> FUSB302_INT
- U6 pad 12: unconnected-(U6-GPIO9-Pad12) -> Npxl
- U6 pad 13: unconnected-(U6-GPIO10-Pad13) -> EC_GP10
- U6 pad 14: unconnected-(U6-GPIO11-Pad14) -> EC_GP11
- U6 pad 24: unconnected-(U6-SWCLK-Pad24) -> Net-(J21-Pin_3)
- U6 pad 25: unconnected-(U6-SWD-Pad25) -> Net-(J21-Pin_2)
- U6 pad 27: unconnected-(U6-GPIO16-Pad27) -> CHG_PWR
- U6 pad 28: unconnected-(U6-GPIO17-Pad28) -> CHG_DIS
- U6 pad 29: unconnected-(U6-GPIO18-Pad29) -> PI_PWR_EN
- U6 pad 30: unconnected-(U6-GPIO19-Pad30) -> EC_GP19
- U6 pad 31: unconnected-(U6-GPIO20-Pad31) -> EC_GP20
- U6 pad 32: unconnected-(U6-GPIO21-Pad32) -> EC_GP21
- U6 pad 34: unconnected-(U6-GPIO22-Pad34) -> EC_GP22
- U6 pad 35: unconnected-(U6-GPIO23-Pad35) -> EC_GP23
- U6 pad 36: unconnected-(U6-GPIO24-Pad36) -> EC_GP24
- U6 pad 37: unconnected-(U6-GPIO25-Pad37) -> EC_GP25
- U8 pad 1: Net-(U8-IO1) -> /USBc_DN
- U8 pad 10: Net-(U8-IO1) -> /USBc_DN
- U8 pad 2: Net-(U8-IO2) -> /USBc_DP
- U8 pad 4: Net-(U8-IO3) -> /USBb_DN
- U8 pad 5: Net-(U8-IO4) -> /USBb_DP
- U8 pad 6: Net-(U8-IO4) -> /USBb_DP
- U8 pad 7: Net-(U8-IO3) -> /USBb_DN
- U8 pad 9: Net-(U8-IO2) -> /USBc_DP
Routing:
- net +5VD: track 0.00 -> 221.3 mm, vias 0 -> 7
- net EC_HwSDA: track 6.40 -> 216.6 mm, vias 0 -> 6
- net EC_HwSCL: track 4.82 -> 214.9 mm, vias 0 -> 8
- net Pi_HwSDA: track 0.00 -> 183.2 mm, vias 0 -> 2
- net Pi_HwSCL: track 0.00 -> 177.1 mm, vias 0 -> 2
- net +3V3: track 66.0 -> 224.0 mm, vias 2 -> 9
- net INT: track 0.00 -> 142.6 mm, vias 0 -> 1
- net +3V3E: track 122.8 -> 264.6 mm, vias 4 -> 17
- net FUSB302_INT: track 0.00 -> 128.5 mm, vias 0 -> 2
- net /Npxl2: track 0.00 -> 119.4 mm, vias 0 -> 4
- net S0I: track 0.00 -> 98.2 mm, vias 0 -> 1
- net S0E1: track 0.00 -> 91.0 mm, vias 0 -> 1
- net S0O: track 0.00 -> 88.7 mm, vias 0 -> 1
- net S0C: track 0.00 -> 88.4 mm, vias 0 -> 1
- net S0E0: track 0.00 -> 87.9 mm, vias 0 -> 1
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- added copper zone on In1.Cu, net GND
- added copper zone on In2.Cu, net GND
Other:
- outline, holes or cut-outs redrawn
- copper layers 2 -> 4
- board text added: "(SDIO)"
- board text added: "- modular power management - USB-C DRP - RP2040 EC - mPCIe 4G - modular IO (screen & user controls) - OLED & keypad header (dbg) - ESP32 WiFi/BT"
- board text added: "ESP32 -C6 WiFi BT ZigBee"
- board text added: "JST"
- board text added: "OLED"
- board text added: "Project funded by"
- board text added: "USB-C"
- board text added: "ZeroPhone Next development board v0"
- board text added: "audio codec goes here"
- board text added: "croc clip goes here"
- board text added: "funded by"
- board text added: "future:"
- board text added: "wifi ant cutout?"
- board text removed: "ESP32 WiFi"
- board text removed: "audio codec"
- board text removed: "copper pad"
- board text removed: "wifi ant cutout"
