File: Raspberry Pi stuff/zpui_businesscard/zpui_businesscard.kicad_pcb (KiCad board)
At the start: 2 copper layers, 89 x 51.3 mm, 34 parts, among them J1 Sn, J2 Se, J3 Ss, J4 Sw, J5 Raspberry_Pi_2_3, J7 I2C, J8 QWIIC, J9 QWIIC, SW1 PgDn, SW10 Down, SW11 Right, SW12 Left, SW2 Scrt, SW7 PgUp, SW8 Ok, SW9 Up, U4 PCF8574

Commit message: zpui_businesscard: v1
Other:
- board text added: "Development funded by"
- board text removed: "ZPUI shield"
